Commit message: its working!

File: src/carbot_hardware/description/ros2_control/carlikebot.ros2_control.xacro (robot description, xacro)
@@ -45,6 +45,6 @@
           <plugin>gazebo_ros2_control/GazeboSystem</plugin>
         </hardware>
-        <!-- drive joint -->
-        <joint name="${prefix}virtual_rear_wheel_joint">
+        <!-- front left -->
+        <joint name="${prefix}front_left_wheel_joint">
           <command_interface name="velocity">
             <param name="min">-1000</param>
@@ -61,7 +61,10 @@
           </state_interface>
         </joint>
-        <joint name="${prefix}rear_left_wheel_joint">
-          <param name="mimic">virtual_rear_wheel_joint</param>
-          <param name="multiplier">${speed_multiplier}</param>
+        <!-- front right -->
+        <joint name="${prefix}front_right_wheel_joint">
+          <command_interface name="velocity">
+            <param name="min">-1000</param>
+            <param name="max">1000</param>
+          </command_interface>
           <state_interface name="velocity">
             <param name="initial_value">0.0</param>
@@ -74,7 +77,10 @@
           </state_interface>
         </joint>
-        <joint name="${prefix}rear_right_wheel_joint">
-          <param name="mimic">virtual_rear_wheel_joint</param>
-          <param name="multiplier">${speed_multiplier}</param>
+        <!-- rear left -->
+        <joint name="${prefix}rear_left_wheel_joint">
+          <command_interface name="velocity">
+            <param name="min">-1000</param>
+            <param name="max">1000</param>
+          </command_interface>
           <state_interface name="velocity">
             <param name="initial_value">0.0</param>
@@ -87,56 +93,13 @@
           </state_interface>
         </joint>
-        <!-- steer joint -->
-        <joint name="${prefix}virtual_front_wheel_joint">
-          <command_interface name="position">
+        <!-- rear right -->
+        <joint name="${prefix}rear_right_wheel_joint">
+          <command_interface name="velocity">
             <param name="min">-1000</param>
             <param name="max">1000</param>
           </command_interface>
-          <state_interface name="position">
-            <param name="initial_value">0.0</param>
-          </state_interface>
-          <state_interface name="effort">
-            <param name="initial_value">0.0</param>
-          </state_interface>
-        </joint>
-        <joint name="${prefix}front_right_wheel_joint">
-          <param name="mimic">virtual_rear_wheel_joint</param>
-          <param name="multiplier">${speed_multiplier}</param>
           <state_interface name="velocity">
             <param name="initial_value">0.0</param>
           </state_interface>
-          <state_interface name="position">
-            <param name="initial_value">0.0</param>
-          </state_interface>
-          <state_interface name="effort">
-            <param name="initial_value">0.0</param>
-          </state_interface>
-        </joint>
-        <joint name="${prefix}front_left_wheel_joint">
-          <param name="mimic">virtual_rear_wheel_joint</param>
-          <param name="multiplier">${speed_multiplier}</param>
-          <state_interface name="velocity">
-            <param name="initial_value">0.0</param>
-          </state_interface>
-          <state_interface name="position">
-            <param name="initial_value">0.0</param>
-          </state_interface>
-          <state_interface name="effort">
-            <param name="initial_value">0.0</param>
-          </state_interface>
-        </joint>
-        <joint name="${prefix}front_left_steer_joint">
-          <param name="mimic">virtual_front_wheel_joint</param>
-          <param name="multiplier">1</param>
-          <state_interface name="position">
-            <param name="initial_value">0.0</param>
-          </state_interface>
-          <state_interface name="effort">
-            <param name="initial_value">0.0</param>
-          </state_interface>
-        </joint>
-        <joint name="${prefix}front_right_steer_joint">
-          <param name="mimic">virtual_front_wheel_joint</param>
-          <param name="multiplier">1</param>
           <state_interface name="position">
             <param name="initial_value">0.0</param>

File: src/carbot_hardware/description/urdf/bigbrain.urdf.xacro (robot description, xacro)
@@ -5,31 +5,30 @@
   <xacro:property name="PI" value="3.1415926535897931"/>
   <xacro:property name="base_mass" value="10" /> <!-- arbitrary value for base mass -->
-  <xacro:property name="base_width" value="0.1351" />
-  <xacro:property name="base_length" value="0.1778" />
-  <xacro:property name="base_height" value="0.030" />
-  <xacro:property name="wheelbase" value="0.1778" />
+  <xacro:property name="base_width" value="0.240" />
+  <xacro:property name="base_length" value="0.300" />
+  <xacro:property name="base_height" value="0.140" />
+  <xacro:property name="wheelbase" value=".2845" />
+  <xacro:property name="wheel_width" value="0.0265" />
+  <xacro:property name="wheel_radius" value="0.032" />
   <xacro:property name="wheel_mass" value="0.34055" /> <!-- arbitrary value for wheel mass -->
-  <xacro:property name="wheel_len" value="0.03" />
-  <xacro:property name="wheel_radius" value="0.0375" />
-  <xacro:property name="wheeltrack" value=".1651"/>
   <xacro:property name="friction" value="3"/>
   <xacro:property name="damping" value="0.01"/>
   <!-- ======================================================================================== -->
   <!-- Base Link -->
-  <link name="${prefix}base_link" />
+  <link name="${prefix}base_link"/>
   <!-- Chassis -->
   <link name="${prefix}chassis_link">
-    <!-- <collision>
-      <origin xyz="0 0 0" rpy="0 0 0"/>
+    <collision>
+      <origin xyz="0 0 0" rpy="0 0 ${PI/2}"/>
       <geometry>
-        <box size="${base_length} ${base_width} ${base_height}"/>
+        <mesh filename="file://$(find carbot_hardware)/urdf/assets/Chassis.stl"/>
       </geometry>
-    </collision> -->
+    </collision>
     <visual>
-      <origin xyz="0 0 0" rpy="0 0 0"/>
+      <origin xyz="0 0 0" rpy="0 0 ${PI/2}"/>
       <geometry>
-        <box size="${base_length} ${base_width} ${base_height}"/>
+        <mesh filename="file://$(find carbot_hardware)/urdf/assets/Chassis.stl"/>
       </geometry>
-      <material name="orange"/>
+      <material name="grey"/>
     </visual>
     <inertial>
@@ -43,22 +42,23 @@
   </link>
     <gazebo reference="chassis_link">
-      <material>Gazebo/Orange</material>
+      <material>Gazebo/Grey</material>
     </gazebo>
     <joint name="${prefix}chassis_joint" type="fixed">
       <parent link="${prefix}base_link"/>
       <child link="${prefix}chassis_link"/>
-      <origin xyz="0 0 ${base_height/2 + wheel_radius}" rpy="0 0 0"/>
+      <origin xyz="0 0 ${.0199 + wheel_radius}" rpy="0 0 0"/>
       <axis xyz="0 0 1"/>
       <dynamics damping="${damping}"/>
     </joint>
     <!-- ==================================================================== -->
-    <xacro:macro name="rear_wheel" params="name x y z direction">
+    <xacro:macro name="wheel" params="name x y z front side">
         <link name="${name}_wheel">
+            <!-- COLLISION -->
             <collision>
-                <origin xyz="0 0 0" rpy="${PI/2} 0 ${PI/2}"/>
-                <geometry>
-                  <cylinder length="${wheel_len}" radius="${wheel_radius}"/>
-                </geometry>
-                <surface>
+              <origin xyz="0 0 0" rpy="${side * -PI/2} 0 0"/>
+              <geometry>
+                <mesh filename="file://$(find carbot_hardware)/urdf/assets/Wheel.stl"/>
+              </geometry>
+              <surface>
                   <friction>
                     <ode>
@@ -69,11 +69,13 @@
                 </surface>
             </collision>
+            <!-- VISIUAL -->
             <visual>
-                <origin xyz="0 0 0" rpy="${PI/2} 0 ${PI/2}"/>
+                <origin xyz="0 0 0" rpy="${side * -PI/2} 0 0"/>
                 <geometry>
-                    <cylinder length="${wheel_len}" radius="${wheel_radius}"/>
+                    <mesh filename="file://$(find carbot_hardware)/urdf/assets/Wheel.stl"/>
                 </geometry>
                 <material name="black"/>
             </visual>
+            <!-- INERTIAL -->
             <inertial>
                 <origin xyz="0 0 0" rpy="${PI/2} 0 ${PI/2}"/>
@@ -87,142 +89,20 @@
         <gazebo reference="${name}_wheel">
             <material>Gazebo/Black</material>
-          </gazebo>
+        </gazebo>
         <joint name="${name}_wheel_joint" type="continuous">
             <parent link="${prefix}chassis_link"/>
             <child link="${name}_wheel"/>
-            <origin xyz="-${wheelbase/2} ${base_width/2 * direction} -${base_height/2}" rpy="0 0 ${PI/2}"/>
-            <axis xyz="1 0 0"/>
+            <origin xyz="${front * .120} ${side * .129} -.0199" rpy="0 0 0"/>
+            <axis xyz="0 1 0"/>
             <limit effort="1000.0" velocity="100.0"/>
             <dynamics damping="${damping}"/>
-            <mimic joint="${prefix}virtual_rear_wheel_joint" multiplier="1.0" offset="0.0"/>
-        </joint>
-    </xacro:macro>
-    <!-- =================================================================================================== -->
-    <xacro:macro name="front_wheel" params="name x y z direction">
-        <link name="${name}_wheel">
-            <collision>
-                <origin xyz="0 0 0" rpy="0 ${PI/2} 0"/>
-                <geometry>
-                  <cylinder length="${wheel_len}" radius="${wheel_radius}"/>
-                </geometry>
-                <surface>
-                  <friction>
-                    <ode>
-                      <mu value="${friction}"/>
-                      <mu2 value="${friction}"/>
-                    </ode>
-                  </friction>
-                </surface>
-            </collision>
-            <visual>
-                <origin xyz="0 0 0" rpy="0 ${PI/2} 0"/>
-                <geometry>
-                    <cylinder length="${wheel_len}" radius="${wheel_radius}"/>
-                </geometry>
-                <material name="black"/>
-            </visual>
-            <inertial>
-                <origin xyz="0 0 0" rpy="0 ${PI/2} 0"/>
-                <mass value="${wheel_mass}"/>
-                <inertia
-                    ixx="0.000270" ixy="0.0" ixz="0.0"
-                    iyy="0.000270" iyz="0.0"
-                    izz="0.000426"/>
-            </inertial>
-        </link>
-        <link name="${name}_steer">
-            <inertial>
-                <origin xyz="0 0 0" rpy="${PI/2} 0 ${PI/2}"/>
-                <mass value="${wheel_mass}"/>
-                <inertia
-                    ixx="0.000270" ixy="0.0" ixz="0.0"
-                    iyy="0.000270" iyz="0.0"
-                    izz="0.000426"/>
-            </inertial>
-        </link>
-        <gazebo reference="${name}_wheel">
-            <material>Gazebo/Black</material>
-          </gazebo>
-        <joint name="${name}_wheel_joint" type="continuous">
-            <parent link="${name}_steer"/>
-            <child link="${name}_wheel"/>
-            <origin xyz="0 0 0" rpy="0 0 0"/>
-            <axis xyz="1 0 0"/>
-            <limit effort="100.0" velocity="100.0"/>
-            <dynamics damping="${damping}"/>
-            <mimic joint="${prefix}virtual_rear_wheel_joint" multiplier="1.0" offset="0.0"/>
-        </joint>
-        <joint name="${name}_steer_joint" type="revolute">
-            <parent link="${prefix}chassis_link"/>
-            <child link="${name}_steer"/>
-            <origin xyz="${wheelbase/2} ${base_width/2 * direction} -${base_height/2}" rpy="0 0 ${PI/2}"/>
-            <axis xyz="0 0 1"/>
-            <limit lower="-0.5" upper="0.5" effort="1000.0" velocity="0.0000001"/>
-            <dynamics damping="${damping}"/>
-            <mimic joint="${prefix}virtual_front_wheel_joint" multiplier="1.0" offset="0.0"/>
+            <!-- <mimic joint="${prefix}virtual_rear_wheel_joint" multiplier="1.0" offset="0.0"/> -->
         </joint>
     </xacro:macro>
     <!-- ====================================================================================================== -->
-    <xacro:front_wheel name="front_left" x="0" y="0" z="0" direction="-1"/>
-    <xacro:front_wheel name="front_right" x="0" y="0" z="0" direction="1"/>
-    <xacro:rear_wheel name="rear_left" x="0" y="0" z="0" direction="-1"/>
-    <xacro:rear_wheel name="rear_right" x="0" y="0" z="0" direction="1"/>
-    <!-- virtual rear wheel -->
-    <link name="${prefix}virtual_rear_wheel">
-      <!-- <visual>
-        <origin xyz="0 0 0" rpy="${PI/2} 0 ${PI/2}"/>
-        <geometry>
-          <cylinder length="0.01" radius="${wheel_radius}"/>
-        </geometry>
-        <material name="invisible"/>
-      </visual> -->
-      <inertial>
-        <origin xyz="0 0 0" rpy="${PI/2} 0 ${PI/2}"/>
-        <mass value="${wheel_mass}"/>
-        <inertia
-          ixx="0.000270" ixy="0.0" ixz="0.0"
-          iyy="0.000270" iyz="0.0"
-          izz="0.000426"/>
-      </inertial>
-    </link>
-    <gazebo reference="${prefix}virtual_rear_wheel">
-      <material>Gazebo/Black</material>
-    </gazebo>
-    <joint name="${prefix}virtual_rear_wheel_joint" type="continuous">
-      <parent link="${prefix}chassis_link"/>
-      <child link="${prefix}virtual_rear_wheel"/>
-      <origin xyz="-${wheelbase/2} 0 -${base_height/2}" rpy="0 0 ${PI/2}"/>
-      <axis xyz="1 0 0"/>
-      <limit effort="100.0" velocity="100.0"/>
-      <dynamics damping="${damping}"/>
-    </joint>
-    <link name="${prefix}virtual_front_wheel">
-      <!-- <visual>
-        <origin xyz="0 0 0" rpy="${PI/2} 0 ${PI/2}"/>
-        <geometry>
-          <cylinder length="0.01" radius="${wheel_radius}"/>
-        </geometry>
-        <material name="invisible"/>
-      </visual> -->
-      <inertial>
-        <origin xyz="0 0 0" rpy="${PI/2} 0 ${PI/2}"/>
-        <mass value="${wheel_mass}"/>
-        <inertia
-          ixx="0.000270" ixy="0.0" ixz="0.0"
-          iyy="0.000270" iyz="0.0"
-          izz="0.000426"/>
-      </inertial>
-    </link>
-    <gazebo reference="${prefix}virtual_front_wheel">
-      <material>Gazebo/Black</material>
-    </gazebo>
-    <joint name="${prefix}virtual_front_wheel_joint" type="revolute">
-      <parent link="${prefix}chassis_link"/>
-      <child link="${prefix}virtual_front_wheel"/>
-      <origin xyz="${wheelbase/2} 0 -${base_height/2}" rpy="0 0 ${PI/2}"/>
-      <axis xyz="0 0 1"/>
-      <limit lower="-0.4" upper="0.4" effort="100.0" velocity="100.0"/>
-      <dynamics damping="${damping}"/>
-    </joint>
+    <xacro:wheel name="front_left" x="0" y="0" z="0" front="1" side="1"/>
+    <xacro:wheel name="front_right" x="0" y="0" z="0" front="1" side="-1"/>
+    <xacro:wheel name="rear_left" x="0" y="0" z="0" front="-1" side="1"/>
+    <xacro:wheel name="rear_right" x="0" y="0" z="0" front="-1" side="-1"/>
   </xacro:macro>
 </robot>

File: src/carbot_hardware/description/urdf/carlikebot.materials.xacro (robot description, xacro)
@@ -15,5 +15,5 @@
   </material>
   <material name="grey">
-    <color rgba="0.2 0.2 0.2 1.0"/>
+    <color rgba="0.6 0.6 0.6 1.0"/>
   </material>
   <material name="orange">

File: src/carbot_hardware/description/urdf/carlikebot.urdf.xacro (robot description, xacro)
@@ -5,5 +5,4 @@
   <xacro:arg name="sim_mode" default="false"/>
   <!-- Import Robot Description -->
-  <!-- <xacro:include filename="$(find carbot_hardware)/urdf/carlikebot_description.urdf.xacro" /> -->
   <xacro:include filename="$(find carbot_hardware)/urdf/bigbrain.urdf.xacro" />
   <!-- Import Rviz colors -->
@@ -15,10 +14,10 @@
   <!-- <xacro:include filename="$(find carbot_hardware)/urdf/camera.xacro" /> -->
   <!-- Import Depth Camera -->
-  <xacro:include filename="$(find carbot_hardware)/urdf/depth_camera.xacro" />
+  <!-- <xacro:include filename="$(find carbot_hardware)/urdf/depth_camera.xacro" /> -->
   <!-- Import LiDAR -->
-  <xacro:include filename="$(find carbot_hardware)/urdf/lidar.xacro" />
+  <!-- <xacro:include filename="$(find carbot_hardware)/urdf/lidar.xacro" /> -->
   <xacro:carlikebot prefix="$(arg prefix)" />
-  <xacro:camera prefix="$(arg prefix)"/>
-  <xacro:lidar prefix="$(arg prefix)"/>
+  <!-- <xacro:camera prefix="$(arg prefix)"/> -->
+  <!-- <xacro:lidar prefix="$(arg prefix)"/> -->
   <xacro:carlikebot_ros2_control name="CarlikeBot" prefix="$(arg prefix)" />
 </robot>
