Commit message: cleaned up urdf

File: src/carbot_hardware/description/urdf/carlikebot.urdf.xacro (robot description, xacro)
@@ -4,6 +4,8 @@
   <xacro:arg name="prefix" default="" />
   <xacro:arg name="sim_mode" default="false"/>
+  <!-- Import Constants -->
+  <xacro:include filename="$(find carbot_hardware)/urdf/constants.xacro" />
   <!-- Import Robot Description -->
-  <xacro:include filename="$(find carbot_hardware)/urdf/bigbrain.urdf.xacro" />
+  <xacro:include filename="$(find carbot_hardware)/urdf/main.urdf.xacro" />
   <!-- Import Rviz colors -->
   <xacro:include filename="$(find carbot_hardware)/urdf/carlikebot.materials.xacro" />
@@ -16,8 +18,8 @@
   <!-- <xacro:include filename="$(find carbot_hardware)/urdf/depth_camera.xacro" /> -->
   <!-- Import LiDAR -->
-  <!-- <xacro:include filename="$(find carbot_hardware)/urdf/lidar.xacro" /> -->
+  <xacro:include filename="$(find carbot_hardware)/urdf/lidar.xacro" />
   <xacro:carlikebot prefix="$(arg prefix)" />
   <!-- <xacro:camera prefix="$(arg prefix)"/> -->
-  <!-- <xacro:lidar prefix="$(arg prefix)"/> -->
+  <xacro:lidar prefix="$(arg prefix)"/>
   <xacro:carlikebot_ros2_control name="CarlikeBot" prefix="$(arg prefix)" />
 </robot>

File: src/carbot_hardware/description/urdf/lidar.xacro (robot description, xacro)
@@ -4,13 +4,12 @@
         <xacro:property name="x_transform" value="0"/>
         <xacro:property name="y_transform" value="0"/>
-        <xacro:property name="z_transform" value="0.05"/>
-        <xacro:property name="r_transform" value="0"/>
-        <xacro:property name="p_transform" value="0"/>
-        <xacro:property name="y_transform" value="0"/>
-        <xacro:property name="PI" value="3.1415926535897931"/>
+        <xacro:property name="z_transform" value="${0.140 + 0.01}"/>
+        <xacro:property name="roll_transform" value="0"/>
+        <xacro:property name="pitch_transform" value="0"/>
+        <xacro:property name="yaw_transform" value="0"/>
         <joint name="laser_joint" type="fixed">
             <parent link="${prefix}chassis_link"/>
             <child link="${prefix}laser_frame"/>
-            <origin xyz="${x_transform} ${y_transform} ${z_transform}" rpy="${r_transform} ${p_transform} ${y_transform}"/>
+            <origin xyz="${x_transform} ${y_transform} ${base_height}" rpy="${roll_transform} ${pitch_transform} ${yaw_transform}"/>
         </joint>
         <link name="${prefix}laser_frame">
@@ -26,5 +25,5 @@
             <sensor name="laser" type="ray">
                 <pose> 0 0 0 0 0 0 </pose>
-                <visualize>true</visualize>
+                <visualize>false</visualize>
                 <update_rate>20</update_rate>
                 <ray>
