Commit message: build works

File: src/microros_hardware_interface/description/ros2_control/carlikebot.ros2_control.xacro (robot description, xacro)
@@ -2,39 +2,29 @@
 <robot xmlns:xacro="http://www.ros.org/wiki/xacro">
   <xacro:macro name="carlikebot_ros2_control" params="name prefix">
-  <xacro:property name="speed_multiplier" value="1"/>
+  <xacro:macro name="motor" params="name">
+    <joint name="${prefix}name">
+      <command_interface name="velocity">
+        <param name="min">-1000</param>
+        <param name="max">1000</param>
+      </command_interface>
+      <state_interface name="velocity"/>
+      <state_interface name="position"/>
+      <state_interface name="effort"/>
+    </joint>
+  </xacro:macro>
     <xacro:unless value="$(arg sim_mode)">
       <ros2_control name="${name}" type="system">
         <hardware>
           <plugin>microros_hardware_interface/MicroSystemHardware</plugin>
-          <param name="example_param_hw_start_duration_sec">0</param>
-          <param name="example_param_hw_stop_duration_sec">3.0</param>
-          <param name="port">/dev/ttyUSB0</param>
-          <param name="drive_id">virtual_rear_wheel_joint</param>
-          <param name="steer_id">virtual_front_wheel_joint</param>
-          <param name="voltage_sensor_id">voltage_sensor</param>
-          <param name="heartbeat_id">heartbeat</param>
-          <param name="baud_rate">115200</param>
-          <param name="loop_rate">60</param>
-          <param name="timeout_ms">0</param>
+          <param name="front_left_name">front_left_motor</param>
+          <param name="front_right_name">front_right_motor</param>
+          <param name="rear_left_name">rear_left_motor</param>
+          <param name="rear_right_name">rear_right_motor</param>
+          <param name="conversion">1</param>
         </hardware>
-        <joint name="${prefix}virtual_rear_wheel_joint">
-          <command_interface name="velocity"/>
-          <state_interface name="velocity"/>
-          <state_interface name="position"/>
-          <state_interface name="effort"/>
-        </joint>
-        <joint name="${prefix}virtual_front_wheel_joint">
-          <command_interface name="position"/>
-          <state_interface name="position"/>
-          <state_interface name="effort"/>
-        </joint>
-        <sensor name="${prefix}heartbeat">
-          <state_interface name="raw"/>
-          <state_interface name="latency"/>
-          <state_interface name="hertz"/>
-        </sensor>
-        <sensor name="${prefix}voltage_sensor">
-          <state_interface name="voltage"/>
-        </sensor>
+        <xacro:motor name="front_left_wheel_joint"/>
+        <xacro:motor name="front_right_wheel_joint"/>
+        <xacro:motor name="rear_left_wheel_joint"/>
+        <xacro:motor name="rear_right_wheel_joint"/>
       </ros2_control>
     </xacro:unless>
@@ -45,68 +35,8 @@
           <plugin>gazebo_ros2_control/GazeboSystem</plugin>
         </hardware>
-        <!-- front left -->
-        <joint name="${prefix}front_left_wheel_joint">
-          <command_interface name="velocity">
-            <param name="min">-1000</param>
-            <param name="max">1000</param>
-          </command_interface>
-          <state_interface name="velocity">
-            <param name="initial_value">0.0</param>
-          </state_interface>
-          <state_interface name="position">
-            <param name="initial_value">0.0</param>
-          </state_interface>
-          <state_interface name="effort">
-            <param name="initial_value">0.0</param>
-          </state_interface>
-        </joint>
-        <!-- front right -->
-        <joint name="${prefix}front_right_wheel_joint">
-          <command_interface name="velocity">
-            <param name="min">-1000</param>
-            <param name="max">1000</param>
-          </command_interface>
-          <state_interface name="velocity">
-            <param name="initial_value">0.0</param>
-          </state_interface>
-          <state_interface name="position">
-            <param name="initial_value">0.0</param>
-          </state_interface>
-          <state_interface name="effort">
-            <param name="initial_value">0.0</param>
-          </state_interface>
-        </joint>
-        <!-- rear left -->
-        <joint name="${prefix}rear_left_wheel_joint">
-          <command_interface name="velocity">
-            <param name="min">-1000</param>
-            <param name="max">1000</param>
-          </command_interface>
-          <state_interface name="velocity">
-            <param name="initial_value">0.0</param>
-          </state_interface>
-          <state_interface name="position">
-            <param name="initial_value">0.0</param>
-          </state_interface>
-          <state_interface name="effort">
-            <param name="initial_value">0.0</param>
-          </state_interface>
-        </joint>
-        <!-- rear right -->
-        <joint name="${prefix}rear_right_wheel_joint">
-          <command_interface name="velocity">
-            <param name="min">-1000</param>
-            <param name="max">1000</param>
-          </command_interface>
-          <state_interface name="velocity">
-            <param name="initial_value">0.0</param>
-          </state_interface>
-          <state_interface name="position">
-            <param name="initial_value">0.0</param>
-          </state_interface>
-          <state_interface name="effort">
-            <param name="initial_value">0.0</param>
-          </state_interface>
-        </joint>
+        <xacro:motor name="front_left_wheel_joint"/>
+        <xacro:motor name="front_right_wheel_joint"/>
+        <xacro:motor name="rear_left_wheel_joint"/>
+        <xacro:motor name="rear_right_wheel_joint"/>
       </ros2_control>
       <gazebo>

File: src/microros_hardware_interface/description/urdf/core.urdf.xacro (robot description, xacro)
@@ -1,5 +1,5 @@
 <?xml version="1.0"?>
 <!-- 4 Wheel Robot with front steering and rear drive -->
-<robot xmlns:xacro="http://www.ros.org/wiki/xacro" name="carlikebot_robot">
+<robot xmlns:xacro="http://www.ros.org/wiki/xacro" name="microros_hardware">
   <xacro:arg name="prefix" default="" />
   <xacro:arg name="sim_mode" default="false"/>
