Commit message: repeatable error

File: src/microros_hardware_interface/description/ros2_control/microros_hardware.ros2_control.xacro (robot description, xacro)
@@ -1,7 +1,7 @@
 <?xml version="1.0"?>
 <robot xmlns:xacro="http://www.ros.org/wiki/xacro">
-  <xacro:macro name="carlikebot_ros2_control" params="name prefix">
+  <xacro:macro name="micro_system_hardware_ros2_control" params="name prefix">
   <xacro:macro name="motor" params="name">
-    <joint name="${prefix}name">
+    <joint name="${name}">
       <command_interface name="velocity">
         <param name="min">-1000</param>
@@ -17,9 +17,19 @@
         <hardware>
           <plugin>microros_hardware_interface/MicroSystemHardware</plugin>
-          <param name="front_left_name">front_left_motor</param>
-          <param name="front_right_name">front_right_motor</param>
-          <param name="rear_left_name">rear_left_motor</param>
-          <param name="rear_right_name">rear_right_motor</param>
-          <param name="conversion">1</param>
+          <!-- Joint Names -->
+          <param name="front_left_joint">front_left_joint</param>
+          <param name="front_right_joint">front_right_joint</param>
+          <param name="rear_left_joint">rear_left_joint</param>
+          <param name="rear_right_joint">rear_right_joint</param>
+          <!-- Topic Names -->
+          <param name="front_left_topic">front_left_motor</param>
+          <param name="front_right_topic">front_right_motor</param>
+          <param name="rear_left_topic">rear_left_motor</param>
+          <param name="rear_right_topic">rear_right_motor</param>
+          <!-- Conversions -->
+          <param name="front_left_conversion">1</param>
+          <param name="front_right_conversion">1</param>
+          <param name="rear_left_conversion">1</param>
+          <param name="rear_right_conversion">1</param>
         </hardware>
         <xacro:motor name="front_left_wheel_joint"/>
@@ -42,5 +52,5 @@
       <gazebo>
         <plugin name="gazebo_ros2_control" filename="libgazebo_ros2_control.so">
-          <parameters>$(find microros_hardware_interface)/bringup/config/carlikebot_controllers.yaml</parameters>
+          <parameters>$(find microros_hardware_interface)/bringup/config/controllers.yaml</parameters>
           <parameters>$(find microros_hardware_interface)/bringup/config/gazebo_controller.yaml</parameters>
         </plugin>

File: src/microros_hardware_interface/description/urdf/core.urdf.xacro (robot description, xacro)
@@ -5,11 +5,11 @@
   <xacro:arg name="sim_mode" default="false"/>
   <!-- Import Constants -->
-  <xacro:include filename="$(find microros_hardware_interface)/urdf/util/constants.xacro" />
+  <xacro:include filename="$(find microros_hardware_interface)/description/urdf/util/constants.xacro" />
   <!-- Import Robot Description -->
-  <xacro:include filename="$(find microros_hardware_interface)/urdf/robot.urdf.xacro" />
+  <xacro:include filename="$(find microros_hardware_interface)/description/urdf/robot.urdf.xacro" />
   <!-- Import Rviz colors -->
-  <xacro:include filename="$(find microros_hardware_interface)/urdf/util/carlikebot.materials.xacro" />
+  <xacro:include filename="$(find microros_hardware_interface)/description/urdf/util/materials.xacro" />
   <!-- Import Hardware Interface -->
-  <xacro:include filename="$(find microros_hardware_interface)/ros2_control/carlikebot.ros2_control.xacro" />
+  <xacro:include filename="$(find microros_hardware_interface)/description/ros2_control/microros_hardware.ros2_control.xacro" />
   <!-- <xacro:include filename="$(find microros_hardware_interface)/ros2_control/sim.xacro"/> -->
   <!-- Import Camera -->
@@ -18,8 +18,8 @@
   <!-- <xacro:include filename="$(find microros_hardware_interface)/urdf/components/depth_camera.xacro" /> -->
   <!-- Import LiDAR -->
-  <xacro:include filename="$(find microros_hardware_interface)/urdf/components/lidar.xacro" />
-  <xacro:carlikebot prefix="$(arg prefix)" />
+  <xacro:include filename="$(find microros_hardware_interface)/description//urdf/components/lidar.xacro" />
+  <xacro:robot_hardware prefix="$(arg prefix)" />
   <!-- <xacro:camera prefix="$(arg prefix)"/> -->
   <xacro:lidar prefix="$(arg prefix)"/>
-  <xacro:carlikebot_ros2_control name="CarlikeBot" prefix="$(arg prefix)" />
+  <xacro:micro_system_hardware_ros2_control name="MicroSystemHardware" prefix="$(arg prefix)" />
 </robot>

File: src/microros_hardware_interface/description/urdf/robot.urdf.xacro (robot description, xacro)
@@ -1,5 +1,5 @@
 <?xml version="1.0"?>
 <robot xmlns:xacro="http://www.ros.org/wiki/xacro">
-  <xacro:macro name="carlikebot" params="prefix">
+  <xacro:macro name="robot_hardware" params="prefix">
     <!-- Base Link -->
     <link name="${prefix}base_link"/>

Commit message: omg it works

File: src/microros_hardware_interface/description/ros2_control/microros_hardware.ros2_control.xacro (robot description, xacro)
@@ -4,5 +4,5 @@
   <xacro:macro name="motor" params="name">
     <joint name="${name}">
-      <command_interface name="effort">
+      <command_interface name="velocity">
         <param name="min">-1000</param>
         <param name="max">1000</param>
@@ -17,4 +17,6 @@
         <hardware>
           <plugin>microros_hardware_interface/MicroSystemHardware</plugin>
+          <!-- Prefix -->
+          <param name="prefix">/esp32</param>
           <!-- Joint Names -->
           <param name="front_left_joint">front_left_wheel_joint</param>

File: src/microros_hardware_interface/description/urdf/robot.urdf.xacro (robot description, xacro)
@@ -9,5 +9,5 @@
         <origin xyz="0 0 0" rpy="0 0 ${PI/2}"/>
         <geometry>
-          <mesh filename="file://$(find microros_hardware_interface)/urdf/assets/Chassis.stl"/>
+          <mesh filename="file://$(find microros_hardware_interface)/description/urdf/assets/Chassis.stl"/>
         </geometry>
       </collision>
@@ -15,5 +15,5 @@
         <origin xyz="0 0 0" rpy="0 0 ${PI/2}"/>
         <geometry>
-          <mesh filename="file://$(find microros_hardware_interface)/urdf/assets/Chassis.stl"/>
+          <mesh filename="file://$(find microros_hardware_interface)/description/urdf/assets/Chassis.stl"/>
         </geometry>
         <material name="grey"/>
@@ -45,5 +45,5 @@
                 <origin xyz="0 0 0" rpy="${side * -PI/2} 0 0"/>
                 <geometry>
-                  <mesh filename="file://$(find microros_hardware_interface)/urdf/assets/Wheel.stl"/>
+                  <mesh filename="file://$(find microros_hardware_interface)/description/urdf/assets/Wheel.stl"/>
                 </geometry>
                 <surface>
@@ -60,5 +60,5 @@
                   <origin xyz="0 0 0" rpy="${side * -PI/2} 0 0"/>
                   <geometry>
-                      <mesh filename="file://$(find microros_hardware_interface)/urdf/assets/Wheel.stl"/>
+                      <mesh filename="file://$(find microros_hardware_interface)/description/urdf/assets/Wheel.stl"/>
                   </geometry>
                   <material name="black"/>

Commit message: removed two wheels, need to fix urdf

File: src/microros_hardware_interface/description/ros2_control/microros_hardware.ros2_control.xacro (robot description, xacro)
@@ -20,26 +20,18 @@
           <param name="prefix">/esp32</param>
           <!-- Joint Names -->
-          <param name="front_left_joint">front_left_wheel_joint</param>
-          <param name="front_right_joint">front_right_wheel_joint</param>
-          <param name="rear_left_joint">rear_left_wheel_joint</param>
-          <param name="rear_right_joint">rear_right_wheel_joint</param>
+          <param name="left_joint">left_wheel_joint</param>
+          <param name="right_joint">right_wheel_joint</param>
           <!-- Topic Names -->
-          <param name="front_left_topic">front_left_motor</param>
-          <param name="front_right_topic">front_right_motor</param>
-          <param name="rear_left_topic">rear_left_motor</param>
-          <param name="rear_right_topic">rear_right_motor</param>
+          <param name="left_topic">left_motor</param>
+          <param name="right_topic">right_motor</param>
           <!-- Conversions -->
           <param name="conversion">0.000294731376096</param>
           <!-- 1 / (2pi * 45 * 12) -->
           <!-- Inverts -->
-          <param name="front_left_inverted">false</param>
-          <param name="front_right_inverted">true</param>
-          <param name="rear_left_inverted">false</param>
-          <param name="rear_right_inverted">true</param>
+          <param name="left_inverted">false</param>
+          <param name="right_inverted">false</param>
         </hardware>
-        <xacro:motor name="front_left_wheel_joint"/>
-        <xacro:motor name="front_right_wheel_joint"/>
-        <xacro:motor name="rear_left_wheel_joint"/>
-        <xacro:motor name="rear_right_wheel_joint"/>
+        <xacro:motor name="left_wheel_joint"/>
+        <xacro:motor name="right_wheel_joint"/>
       </ros2_control>
     </xacro:unless>
@@ -50,8 +42,6 @@
           <plugin>ign_ros2_control/IgnitionSystem</plugin>
         </hardware>
-        <xacro:motor name="front_left_wheel_joint"/>
-        <xacro:motor name="front_right_wheel_joint"/>
-        <xacro:motor name="rear_left_wheel_joint"/>
-        <xacro:motor name="rear_right_wheel_joint"/>
+        <xacro:motor name="left_wheel_joint"/>
+        <xacro:motor name="right_wheel_joint"/>
       </ros2_control>
       <gazebo>

File: src/microros_hardware_interface/description/urdf/core.urdf.xacro (robot description, xacro)
@@ -8,4 +8,5 @@
   <!-- Import Macros -->
   <xacro:include filename="$(find microros_hardware_interface)/description/urdf/util/macros/wheel.xacro" />
+  <xacro:include filename="$(find microros_hardware_interface)/description/urdf/util/macros/dead_wheel.xacro" />
   <xacro:include filename="$(find microros_hardware_interface)/description/urdf/util/macros/camera.xacro" />
   <xacro:include filename="$(find microros_hardware_interface)/description/urdf/util/macros/depth_camera.xacro" />

File: src/microros_hardware_interface/description/urdf/robot.urdf.xacro (robot description, xacro)
@@ -40,8 +40,8 @@
     </joint>
     <!--front is positive, left is positive-->
-    <xacro:wheel name="front_left" x="0" y="0" z="0" front="1" side="1"/>
-    <xacro:wheel name="front_right" x="0" y="0" z="0" front="1" side="-1"/>
-    <xacro:wheel name="rear_left" x="0" y="0" z="0" front="-1" side="1"/>
-    <xacro:wheel name="rear_right" x="0" y="0" z="0" front="-1" side="-1"/>
+    <xacro:wheel name="left" x="0" y="0" z="0" front="-1" side="-1"/>
+    <xacro:wheel name="right" x="0" y="0" z="0" front="-1" side="1"/>
+    <xacro:dead_wheel name="left_caster" x="0" y="0" z="0" front="1" side="-1"/>
+    <xacro:dead_wheel name="right_caster" x="0" y="0" z="0" front="1" side="1"/>
   </xacro:macro>
 </robot>

File: src/microros_hardware_interface/description/urdf/util/constants.xacro (robot description, xacro)
@@ -2,5 +2,5 @@
 <robot xmlns:xacro="http://www.ros.org/wiki/xacro">
     <xacro:property name="PI" value="3.1415926535897931"/>
-    <xacro:property name="base_mass" value="3" /> <!-- arbitrary value for base mass -->
+    <xacro:property name="base_mass" value="1" /> <!-- arbitrary value for base mass -->
     <xacro:property name="base_width" value="0.240" />
     <xacro:property name="base_length" value="0.300" />
@@ -12,4 +12,4 @@
     <xacro:property name="friction" value="1"/>
     <xacro:property name="min_depth" value="0.5"/>
-    <xacro:property name="damping" value="0.1"/>
+    <xacro:property name="damping" value="0.001"/>
 </robot>

File: src/microros_hardware_interface/description/urdf/util/macros/wheel.xacro (robot description, xacro)
@@ -51,7 +51,9 @@
             </inertial>
         </link>
-        <!-- <gazebo reference="${name}_wheel">
+        <gazebo reference="${name}_wheel">
             <material>Gazebo/Black</material>
-        </gazebo> -->
+            <mu1 value="1"/>
+            <mu2 value="1"/>
+        </gazebo>
         <joint name="${name}_wheel_joint" type="continuous">
             <parent link="${prefix}chassis_link"/>
