Commit message: hooray!

File: src/microros_hardware_interface/description/urdf/robot.urdf.xacro (robot description, xacro)
@@ -45,5 +45,6 @@
                 <origin xyz="0 0 0" rpy="${side * -PI/2} 0 0"/>
                 <geometry>
-                  <mesh filename="file://$(find microros_hardware_interface)/description/urdf/assets/Wheel.stl"/>
+                  <!-- <mesh filename="file://$(find microros_hardware_interface)/description/urdf/assets/Wheel.stl"/> -->
+                  <sphere radius="${wheel_radius}" />
                 </geometry>
                 <surface>
@@ -61,4 +62,5 @@
                   <geometry>
                       <mesh filename="file://$(find microros_hardware_interface)/description/urdf/assets/Wheel.stl"/>
+                      <!-- <sphere radius="${wheel_radius}" /> -->
                   </geometry>
                   <material name="black"/>

File: src/microros_hardware_interface/description/urdf/util/constants.xacro (robot description, xacro)
@@ -2,5 +2,5 @@
 <robot xmlns:xacro="http://www.ros.org/wiki/xacro">
     <xacro:property name="PI" value="3.1415926535897931"/>
-    <xacro:property name="base_mass" value="10" /> <!-- arbitrary value for base mass -->
+    <xacro:property name="base_mass" value="1" /> <!-- arbitrary value for base mass -->
     <xacro:property name="base_width" value="0.240" />
     <xacro:property name="base_length" value="0.300" />
@@ -10,5 +10,5 @@
     <xacro:property name="wheel_radius" value="0.032" />
     <xacro:property name="wheel_mass" value="0.34055" /> <!-- arbitrary value for wheel mass -->
-    <xacro:property name="friction" value="3"/>
+    <xacro:property name="friction" value="0.0"/>
     <xacro:property name="damping" value="0.01"/>
 </robot>

Commit message: idk

File: src/microros_hardware_interface/description/urdf/robot.urdf.xacro (robot description, xacro)
@@ -53,6 +53,19 @@
                         <mu value="${friction}"/>
                         <mu2 value="${friction}"/>
+                        <!-- <min_depth value="${min_depth}"/> -->
+                        <!-- <slip1 value="1"/>
+                        <slip2 value="1"/> -->
                       </ode>
+                      <torsional>
+                        <coefficient>0.0</coefficient>
+                      </torsional>
                     </friction>
+                    <contact>
+                      <ode>
+                        <min_depth value="${min_depth}"/>
+                        <!-- <kp>1e15</kp>
+                        <kd>1e13</kd> -->
+                      </ode>
+                    </contact>
                   </surface>
               </collision>

File: src/microros_hardware_interface/description/urdf/util/constants.xacro (robot description, xacro)
@@ -2,5 +2,5 @@
 <robot xmlns:xacro="http://www.ros.org/wiki/xacro">
     <xacro:property name="PI" value="3.1415926535897931"/>
-    <xacro:property name="base_mass" value="1" /> <!-- arbitrary value for base mass -->
+    <xacro:property name="base_mass" value="10" /> <!-- arbitrary value for base mass -->
     <xacro:property name="base_width" value="0.240" />
     <xacro:property name="base_length" value="0.300" />
@@ -10,5 +10,6 @@
     <xacro:property name="wheel_radius" value="0.032" />
     <xacro:property name="wheel_mass" value="0.34055" /> <!-- arbitrary value for wheel mass -->
-    <xacro:property name="friction" value="0.0"/>
+    <xacro:property name="friction" value="100"/>
+    <xacro:property name="min_depth" value="0.5"/>
     <xacro:property name="damping" value="0.01"/>
 </robot>

Commit message: added obj files

File: src/microros_hardware_interface/description/urdf/robot.urdf.xacro (robot description, xacro)
@@ -9,5 +9,5 @@
         <origin xyz="0 0 0" rpy="0 0 ${PI/2}"/>
         <geometry>
-          <mesh filename="file://$(find microros_hardware_interface)/description/urdf/assets/Chassis.stl"/>
+          <mesh filename="file://$(find microros_hardware_interface)/description/urdf/assets/chassis/Chassis.stl"/>
         </geometry>
       </collision>
@@ -15,6 +15,7 @@
         <origin xyz="0 0 0" rpy="0 0 ${PI/2}"/>
         <geometry>
-          <mesh filename="file://$(find microros_hardware_interface)/description/urdf/assets/Chassis.stl"/>
+          <mesh filename="file://$(find microros_hardware_interface)/description/urdf/assets/chassis/Chassis.stl"/>
         </geometry>
+        <cast_shadows>false</cast_shadows>
         <material name="grey"/>
       </visual>
@@ -23,7 +24,7 @@
         <mass value="${base_mass}"/>
           <inertia
-            ixx="0.000270" ixy="0.0" ixz="0.0"
-            iyy="0.000270" iyz="0.0"
-            izz="0.000426"/>
+            ixx="${0.01952332}" ixy="0.0" ixz="0.0"
+            iyy="${0.01450326}" iyz="${-0.00000016}"
+            izz="${0.02678084}"/>
         </inertial>
     </link>
@@ -45,5 +46,5 @@
                 <origin xyz="0 0 0" rpy="${side * -PI/2} 0 0"/>
                 <geometry>
-                  <!-- <mesh filename="file://$(find microros_hardware_interface)/description/urdf/assets/Wheel.stl"/> -->
+                  <!-- <mesh filename="file://$(find microros_hardware_interface)/description/urdf/assets/wheel/Wheel.stl"/> -->
                   <sphere radius="${wheel_radius}" />
                 </geometry>
@@ -74,8 +75,8 @@
                   <origin xyz="0 0 0" rpy="${side * -PI/2} 0 0"/>
                   <geometry>
-                      <mesh filename="file://$(find microros_hardware_interface)/description/urdf/assets/Wheel.stl"/>
+                      <mesh filename="file://$(find microros_hardware_interface)/description/urdf/assets/wheel/Wheel.obj"/>
                       <!-- <sphere radius="${wheel_radius}" /> -->
                   </geometry>
-                  <material name="black"/>
+                  <!-- <material name="black"/> -->
               </visual>
               <!-- INERTIAL -->
@@ -89,7 +90,7 @@
               </inertial>
           </link>
-          <gazebo reference="${name}_wheel">
+          <!-- <gazebo reference="${name}_wheel">
               <material>Gazebo/Black</material>
-          </gazebo>
+          </gazebo> -->
           <joint name="${name}_wheel_joint" type="continuous">
               <parent link="${prefix}chassis_link"/>

File: src/microros_hardware_interface/description/urdf/util/constants.xacro (robot description, xacro)
@@ -2,5 +2,5 @@
 <robot xmlns:xacro="http://www.ros.org/wiki/xacro">
     <xacro:property name="PI" value="3.1415926535897931"/>
-    <xacro:property name="base_mass" value="10" /> <!-- arbitrary value for base mass -->
+    <xacro:property name="base_mass" value="3" /> <!-- arbitrary value for base mass -->
     <xacro:property name="base_width" value="0.240" />
     <xacro:property name="base_length" value="0.300" />
@@ -10,6 +10,6 @@
     <xacro:property name="wheel_radius" value="0.032" />
     <xacro:property name="wheel_mass" value="0.34055" /> <!-- arbitrary value for wheel mass -->
-    <xacro:property name="friction" value="100"/>
+    <xacro:property name="friction" value="1"/>
     <xacro:property name="min_depth" value="0.5"/>
-    <xacro:property name="damping" value="0.01"/>
+    <xacro:property name="damping" value="0.1"/>
 </robot>
