Commit message: checkpoint

File: src/microros_hardware_interface/description/urdf/core.urdf.xacro (robot description, xacro)
@@ -4,6 +4,8 @@
   <xacro:arg name="prefix" default="" />
   <xacro:arg name="sim_mode" default="false"/>
-  <!-- Import Constants -->
+  <!-- Import Static Files -->
   <xacro:include filename="$(find microros_hardware_interface)/description/urdf/util/constants.xacro" />
+  <!-- Import Macros -->
+  <xacro:include filename="$(find microros_hardware_interface)/description/urdf/util/macros/wheel.xacro" />
   <!-- Import Robot Description -->
   <xacro:include filename="$(find microros_hardware_interface)/description/urdf/robot.urdf.xacro" />
@@ -13,16 +15,16 @@
   <xacro:include filename="$(find microros_hardware_interface)/description/ros2_control/microros_hardware.ros2_control.xacro" />
   <xacro:robot_hardware prefix="$(arg prefix)" />
-  <xacro:micro_system_hardware_ros2_control name="MicroSystemHardware" prefix="$(arg prefix)" />
+  <xacro:micro_system_hardware_ros2_control name="MicroSystemHardware" prefix="$(arg prefix)"/>
   <!-- Import Camera -->
-  <xacro:include filename="$(find microros_hardware_interface)/description/urdf/components/camera.xacro" />
+  <xacro:include filename="$(find microros_hardware_interface)/description/urdf/util/components/camera.xacro" />
   <xacro:camera prefix="$(arg prefix)"/>
   <!-- Import Depth Camera -->
-  <xacro:include filename="$(find microros_hardware_interface)/description/urdf/components/depth_camera.xacro" />
+  <xacro:include filename="$(find microros_hardware_interface)/description/urdf/util/components/depth_camera.xacro" />
   <xacro:depth_camera prefix="$(arg prefix)"/>
   <!-- Import LiDAR -->
-  <xacro:include filename="$(find microros_hardware_interface)/description/urdf/components/lidar.xacro" />
+  <xacro:include filename="$(find microros_hardware_interface)/description/urdf/util/components/lidar.xacro" />
   <xacro:lidar prefix="$(arg prefix)"/>
   <!-- Import IMU -->
-  <xacro:include filename="$(find microros_hardware_interface)/description/urdf/components/imu.xacro" />
+  <xacro:include filename="$(find microros_hardware_interface)/description/urdf/util/components/imu.xacro" />
   <xacro:imu prefix="$(arg prefix)"/>
 </robot>

File: src/microros_hardware_interface/description/urdf/robot.urdf.xacro (robot description, xacro)
@@ -29,83 +29,19 @@
         </inertial>
     </link>
-      <gazebo reference="chassis_link">
-        <material>Gazebo/Grey</material>
-      </gazebo>
-      <joint name="${prefix}chassis_joint" type="fixed">
-        <parent link="${prefix}base_link"/>
-        <child link="${prefix}chassis_link"/>
-        <origin xyz="0 0 ${.0199 + wheel_radius}" rpy="0 0 0"/>
-        <axis xyz="0 0 1"/>
-        <dynamics damping="${damping}"/>
-      </joint>
-      <!-- ==================================================================== -->
-      <xacro:macro name="wheel" params="name x y z front side">
-          <link name="${name}_wheel">
-              <!-- COLLISION -->
-              <collision>
-                <origin xyz="0 0 0" rpy="${side * -PI/2} 0 0"/>
-                <geometry>
-                  <!-- <mesh filename="file://$(find microros_hardware_interface)/description/urdf/assets/wheel/Wheel.stl"/> -->
-                  <sphere radius="${wheel_radius}" />
-                </geometry>
-                <surface>
-                    <friction>
-                      <ode>
-                        <mu value="${friction}"/>
-                        <mu2 value="${friction}"/>
-                        <!-- <min_depth value="${min_depth}"/> -->
-                        <!-- <slip1 value="1"/>
-                        <slip2 value="1"/> -->
-                      </ode>
-                      <torsional>
-                        <coefficient>0.0</coefficient>
-                      </torsional>
-                    </friction>
-                    <contact>
-                      <ode>
-                        <min_depth value="${min_depth}"/>
-                        <!-- <kp>1e15</kp>
-                        <kd>1e13</kd> -->
-                      </ode>
-                    </contact>
-                  </surface>
-              </collision>
-              <!-- VISIUAL -->
-              <visual>
-                  <origin xyz="0 0 0" rpy="${side * -PI/2} 0 0"/>
-                  <geometry>
-                      <mesh filename="file://$(find microros_hardware_interface)/description/urdf/assets/wheel/Wheel.obj"/>
-                      <!-- <sphere radius="${wheel_radius}" /> -->
-                  </geometry>
-                  <!-- <material name="black"/> -->
-              </visual>
-              <!-- INERTIAL -->
-              <inertial>
-                  <origin xyz="0 0 0" rpy="${PI/2} 0 ${PI/2}"/>
-                  <mass value="${wheel_mass}"/>
-                  <inertia
-                      ixx="0.000270" ixy="0.0" ixz="0.0"
-                      iyy="0.000270" iyz="0.0"
-                      izz="0.000426"/>
-              </inertial>
-          </link>
-          <!-- <gazebo reference="${name}_wheel">
-              <material>Gazebo/Black</material>
-          </gazebo> -->
-          <joint name="${name}_wheel_joint" type="continuous">
-              <parent link="${prefix}chassis_link"/>
-              <child link="${name}_wheel"/>
-              <origin xyz="${front * .120} ${side * .129} -.0199" rpy="0 0 0"/>
-              <axis xyz="0 1 0"/>
-              <limit effort="1000.0" velocity="100.0"/>
-              <dynamics damping="${damping}"/>
-              <!-- <mimic joint="${prefix}virtual_rear_wheel_joint" multiplier="1.0" offset="0.0"/> -->
-          </joint>
-      </xacro:macro>
-      <!-- ====================================================================================================== -->
-      <xacro:wheel name="front_left" x="0" y="0" z="0" front="1" side="1"/>
-      <xacro:wheel name="front_right" x="0" y="0" z="0" front="1" side="-1"/>
-      <xacro:wheel name="rear_left" x="0" y="0" z="0" front="-1" side="1"/>
-      <xacro:wheel name="rear_right" x="0" y="0" z="0" front="-1" side="-1"/>
+    <gazebo reference="chassis_link">
+      <material>Gazebo/Grey</material>
+    </gazebo>
+    <joint name="${prefix}chassis_joint" type="fixed">
+      <parent link="${prefix}base_link"/>
+      <child link="${prefix}chassis_link"/>
+      <origin xyz="0 0 ${.0199 + wheel_radius}" rpy="0 0 0"/>
+      <axis xyz="0 0 1"/>
+      <dynamics damping="${damping}"/>
+    </joint>
+    <!--front is positive, left is positive-->
+    <xacro:wheel name="front_left" x="0" y="0" z="0" front="1" side="1"/>
+    <xacro:wheel name="front_right" x="0" y="0" z="0" front="1" side="-1"/>
+    <xacro:wheel name="rear_left" x="0" y="0" z="0" front="-1" side="1"/>
+    <xacro:wheel name="rear_right" x="0" y="0" z="0" front="-1" side="-1"/>
   </xacro:macro>
 </robot>

Commit message: checkpoint

File: src/microros_hardware_interface/description/urdf/core.urdf.xacro (robot description, xacro)
@@ -8,4 +8,8 @@
   <!-- Import Macros -->
   <xacro:include filename="$(find microros_hardware_interface)/description/urdf/util/macros/wheel.xacro" />
+  <xacro:include filename="$(find microros_hardware_interface)/description/urdf/util/macros/camera.xacro" />
+  <xacro:include filename="$(find microros_hardware_interface)/description/urdf/util/macros/depth_camera.xacro" />
+  <xacro:include filename="$(find microros_hardware_interface)/description/urdf/util/macros/imu.xacro" />
+  <xacro:include filename="$(find microros_hardware_interface)/description/urdf/util/macros/lidar.xacro" />
   <!-- Import Robot Description -->
   <xacro:include filename="$(find microros_hardware_interface)/description/urdf/robot.urdf.xacro" />
@@ -17,14 +21,16 @@
   <xacro:micro_system_hardware_ros2_control name="MicroSystemHardware" prefix="$(arg prefix)"/>
   <!-- Import Camera -->
-  <xacro:include filename="$(find microros_hardware_interface)/description/urdf/util/components/camera.xacro" />
-  <xacro:camera prefix="$(arg prefix)"/>
+  <!-- <xacro:include filename="$(find microros_hardware_interface)/description/urdf/util/components/camera.xacro" /> -->
+  <!-- <xacro:camera prefix="$(arg prefix)"/> -->
+  <xacro:include filename="$(find microros_hardware_interface)/description/urdf/util/components/driver_camera.xacro" />
   <!-- Import Depth Camera -->
-  <xacro:include filename="$(find microros_hardware_interface)/description/urdf/util/components/depth_camera.xacro" />
-  <xacro:depth_camera prefix="$(arg prefix)"/>
+  <!-- <xacro:include filename="$(find microros_hardware_interface)/description/urdf/util/components/depth_camera.xacro" /> -->
+  <!-- <xacro:depth_camera prefix="$(arg prefix)"/> -->
+  <xacro:camera cam_name="rgbd_camera" namespace="rgbd_camera" parent="chassis_link" x="0.1" y="0" z="0.1" roll="0" pitch="0" yaw="0"/>
   <!-- Import LiDAR -->
-  <xacro:include filename="$(find microros_hardware_interface)/description/urdf/util/components/lidar.xacro" />
-  <xacro:lidar prefix="$(arg prefix)"/>
-  <!-- Import IMU -->
-  <xacro:include filename="$(find microros_hardware_interface)/description/urdf/util/components/imu.xacro" />
-  <xacro:imu prefix="$(arg prefix)"/>
+  <!-- <xacro:include filename="$(find microros_hardware_interface)/description/urdf/util/components/lidar.xacro" />
+  <xacro:lidar prefix="$(arg prefix)"/> -->
+  <xacro:lidar lidar_name="laser" namespace="lidar" parent="chassis_link" x="0" y="0" z="0.14" roll="0" pitch="0" yaw="0"/>
+  <!-- Create IMU -->
+  <xacro:imu imu_name="imu" namespace="imu" parent="chassis_link" x="0.1" y="0" z="0.17" roll="0" pitch="0" yaw="0"/>
 </robot>

File: src/microros_hardware_interface/description/urdf/util/components/camera.xacro (robot description, xacro)
@@ -25,5 +25,5 @@
             <parent link="${prefix}camera_link"/>
             <child link="${prefix}camera_link_optical"/>
-            <origin xyz="${x_transform / 2} ${y_transform} ${z_transform}" rpy="${-PI / 2} 0 ${-PI / 2}"/>
+            <origin xyz="0 0 0" rpy="${-PI / 2} 0 ${-PI / 2}"/>
         </joint>
         <link name="${prefix}camera_link_optical"></link>

File: src/microros_hardware_interface/description/urdf/util/macros/camera.xacro (robot description, xacro)
@@ -1,12 +1,8 @@
 <?xml version="1.0"?>
 <robot xmlns:xacro="http://www.ros.org/wiki/xacro" >
-    <xacro:macro name="camera" params="name parent x y z roll pitch yaw">
+    <xacro:macro name="camera" params="cam_name namespace parent x:=0 y:=0 z:=0 roll:=0 pitch:=0 yaw:=0">
         <xacro:property name="PI" value="3.1415926535897931"/>
-        <joint name="${name}" type="fixed">
-            <parent link="${parent}"/>
-            <child link="${name}_link"/>
-            <origin xyz="${x} ${y} ${z}" rpy="${roll} ${pitch} ${yaw}"/>
-        </joint>
-        <link name="${name}_link">
+        <!-- main link -->
+        <link name="${cam_name}_link">
             <visual>
                 <geometry>
@@ -16,18 +12,30 @@
             </visual>
         </link>
-        <joint name="${name}_optical_joint" type="fixed">
-            <parent link="${name}_link"/>
-            <child link="${name}_link_optical"/>
+        <!-- optical link -->
+        <link name="${cam_name}_link_optical"></link>
+        <!-- main joint -->
+        <joint name="${cam_name}_joint" type="fixed">
+            <parent link="${parent}"/>
+            <child link="${cam_name}_link"/>
+            <origin xyz="${x} ${y} ${z}" rpy="${roll} ${pitch} ${yaw}"/>
+        </joint>
+        <!-- optical joint -->
+        <joint name="${cam_name}_optical_joint" type="fixed">
+            <parent link="${cam_name}_link"/>
+            <child link="${cam_name}_link_optical"/>
             <origin xyz="0 0 0" rpy="${-PI / 2} 0 ${-PI / 2}"/>
         </joint>
-        <link name="${name}camera_link_optical"></link>
-        <gazebo reference="${name}camera_link">
+        <!-- gazebo reference -->
+        <gazebo reference="${cam_name}_link">
             <material>Gazebo/Black</material>
-            <sensor name="camera" type="camera">
+            <sensor name="${namespace}" type="camera">
+                <!-- offset from joint -->
                 <pose> 0 0 0 0 0 0 </pose>
+                <!-- idk what this actually does in new gz -->
                 <visualize>true</visualize>
+                <!-- hz -->
                 <update_rate>30</update_rate>
                 <camera>
-                    <camera_info_topic>camera/camera_info</camera_info_topic>
+                    <!-- <camera_info_topic>${namespace}/camera_info</camera_info_topic> -->
                     <horizontal_fov>1.089</horizontal_fov>
                     <image>
@@ -41,6 +49,6 @@
                     </clip>
                 </camera>
-                <topic>camera/image_raw</topic>
-                <gz_frame_id>camera_link_optical</gz_frame_id>
+                <topic>${namespace}/image_raw</topic>
+                <gz_frame_id>${cam_name}_link_optical</gz_frame_id>
             </sensor>
         </gazebo>

File: src/microros_hardware_interface/description/urdf/util/macros/depth_camera.xacro (robot description, xacro)
@@ -1,18 +1,8 @@
 <?xml version="1.0"?>
 <robot xmlns:xacro="http://www.ros.org/wiki/xacro" >
-    <xacro:macro name="depth_camera" params="prefix">
-        <xacro:property name="x_transform" value="0.1778"/>
-        <xacro:property name="y_transform" value="0"/>
-        <xacro:property name="z_transform" value="0.1"/>
-        <xacro:property name="r_transform" value="0"/>
-        <xacro:property name="p_transform" value="0"/>
-        <xacro:property name="y_transform" value="0"/>
+    <xacro:macro name="depth_camera" params="cam_name namespace parent x:=0 y:=0 z:=0 roll:=0 pitch:=0 yaw:=0">
         <xacro:property name="PI" value="3.1415926535897931"/>
-        <joint name="${prefix}depth_camera_joint" type="fixed">
-            <parent link="${prefix}chassis_link"/>
-            <child link="${prefix}depth_camera_link"/>
-            <origin xyz="${x_transform / 2} ${y_transform} ${z_transform}" rpy="${r_transform} ${p_transform} ${y_transform}"/>
-        </joint>
-        <link name="${prefix}depth_camera_link">
+        <!-- main link -->
+        <link name="${cam_name}_link">
             <visual>
                 <geometry>
@@ -22,16 +12,28 @@
             </visual>
         </link>
-        <joint name="${prefix}depth_camera_optical_joint" type="fixed">
-            <parent link="${prefix}depth_camera_link"/>
-            <child link="${prefix}depth_camera_link_optical"/>
-            <origin xyz="${x_transform / 2} ${y_transform} ${z_transform}" rpy="${-PI / 2} 0 ${-PI / 2}"/>
+        <!-- optical link -->
+        <link name="${cam_name}_link_optical"></link>
+        <!-- main joint -->
+        <joint name="${cam_name}_joint" type="fixed">
+            <parent link="${parent}"/>
+            <child link="${cam_name}_link"/>
+            <origin xyz="${x} ${y} ${z}" rpy="${roll} ${pitch} ${yaw}"/>
         </joint>
-        <link name="${prefix}depth_camera_link_optical"></link>
-        <gazebo reference="${prefix}depth_camera_link">
+        <!-- optical joint -->
+        <joint name="${cam_name}_optical_joint" type="fixed">
+            <parent link="${cam_name}_link"/>
+            <child link="${cam_name}_link_optical"/>
+            <origin xyz="0 0 0" rpy="${-PI / 2} 0 ${-PI / 2}"/>
+        </joint>
+        <gazebo reference="${cam_name}_link">
             <material>Gazebo/Black</material>
-            <sensor name="rgbd_camera" type="rgbd_camera">
+            <sensor name="${namespace}" type="rgbd_camera">
+                <!-- offset from joint -->
                 <pose> 0 0 0 0 0 0 </pose>
+                <!-- idk what this does in new gz -->
                 <visualize>true</visualize>
+                <!-- just keep it on -->
                 <always_on>1</always_on>
+                <!-- hz -->
                 <update_rate>30</update_rate>
                 <camera>
@@ -52,6 +54,6 @@
 					</noise>
                 </camera>
-                <topic>rgbd_camera</topic>
-                <gz_frame_id>depth_camera_link_optical</gz_frame_id>
+                <topic>${namespace}</topic>
+                <gz_frame_id>${cam_name}_link_optical</gz_frame_id>
                 <!-- <plugin filename="RosGzPointCloud" name="ros_gz_point_cloud::PointCloud">
                     <namespace>rgbd_camera</namespace>

File: src/microros_hardware_interface/description/urdf/util/macros/imu.xacro (robot description, xacro)
@@ -1,13 +1,7 @@
 <?xml version="1.0"?>
 <robot xmlns:xacro="http://www.ros.org/wiki/xacro" >
-    <xacro:macro name="imu" params="prefix">
-        <xacro:property name="x_transform" value="0"/>
-        <xacro:property name="y_transform" value="0"/>
-        <xacro:property name="z_transform" value="0.2"/>
-        <xacro:property name="r_transform" value="0"/>
-        <xacro:property name="p_transform" value="0"/>
-        <xacro:property name="y_transform" value="0"/>
+    <xacro:macro name="imu" params="imu_name namespace parent x:=0 y:=0 z:=0 roll:=0 pitch:=0 yaw:=0">
         <xacro:property name="PI" value="3.1415926535897931"/>
-        <link name="${prefix}imu_link">
+        <link name="${imu_name}_link">
             <visual>
                 <geometry>
@@ -17,18 +11,22 @@
             </visual>
         </link>
-        <joint name="${prefix}imu_joint" type="fixed">
-            <parent link="${prefix}chassis_link"/>
-            <child link="${prefix}imu_link"/>
-            <origin xyz="${x_transform / 2} ${y_transform} ${z_transform}" rpy="${r_transform} ${p_transform} ${y_transform}"/>
+        <joint name="${imu_name}_joint" type="fixed">
+            <parent link="${parent}"/>
+            <child link="${imu_name}_link"/>
+            <origin xyz="${x} ${y} ${z}" rpy="${roll} ${pitch} ${yaw}"/>
         </joint>
-        <gazebo reference="${prefix}imu_link">
+        <gazebo reference="${imu_name}_link">
             <material>Gazebo/Black</material>
-            <sensor name="imu" type="imu">
+            <sensor name="${imu_name}" type="imu">
+                <!-- offset from joint -->
                 <pose> 0 0 0 0 0 0 </pose>
+                <!-- idk what this does in new gz -->
                 <visualize>true</visualize>
+                <!-- just keep it on -->
                 <always_on>1</always_on>
+                <!-- hz -->
                 <update_rate>30</update_rate>
-                <topic>imu</topic>
-                <gz_frame_id>imu_link</gz_frame_id>
+                <topic>${namespace}/data</topic>
+                <gz_frame_id>${imu_name}_link</gz_frame_id>
                 <plugin filename="gz-sim-imu-system" name="gz::sim::systems::Imu"/>
             </sensor>

File: src/microros_hardware_interface/description/urdf/util/macros/lidar.xacro (robot description, xacro)
@@ -1,17 +1,11 @@
 <?xml version="1.0"?>
 <robot xmlns:xacro="http://www.ros.org/wiki/xacro" >
-    <xacro:macro name="lidar" params="prefix">
-        <xacro:property name="x_transform" value="0"/>
-        <xacro:property name="y_transform" value="0"/>
-        <xacro:property name="z_transform" value="${0.140 + 0.01}"/>
-        <xacro:property name="roll_transform" value="0"/>
-        <xacro:property name="pitch_transform" value="0"/>
-        <xacro:property name="yaw_transform" value="0"/>
-        <joint name="laser_joint" type="fixed">
-            <parent link="${prefix}chassis_link"/>
-            <child link="${prefix}laser_frame"/>
-            <origin xyz="${x_transform} ${y_transform} ${base_height}" rpy="${roll_transform} ${pitch_transform} ${yaw_transform}"/>
+    <xacro:macro name="lidar" params="lidar_name namespace parent x:=0 y:=0 z:=0 roll:=0 pitch:=0 yaw:=0">
+        <joint name="${lidar_name}_joint" type="fixed">
+            <parent link="${parent}"/>
+            <child link="${lidar_name}_frame"/>
+            <origin xyz="${x} ${y} ${z}" rpy="${roll} ${pitch} ${yaw}"/>
         </joint>
-        <link name="${prefix}laser_frame">
+        <link name="${lidar_name}_frame">
             <visual>
                 <geometry>
@@ -21,9 +15,9 @@
             </visual>
         </link>
-        <gazebo reference="${prefix}laser_frame">
+        <gazebo reference="${lidar_name}_frame">
             <material>Gazebo/Blue</material>
-            <sensor name="laser" type="gpu_lidar">
+            <sensor name="${lidar_name}" type="gpu_lidar">
                 <pose> 0 0 0 0 0 0 </pose>
-                <visualize>false</visualize>
+                <visualize>true</visualize>
                 <update_rate>20</update_rate>
                 <lidar>
@@ -40,6 +34,6 @@
                     </range>
                 </lidar>
-                <topic>scan</topic>
-                <gz_frame_id>laser_frame</gz_frame_id>
+                <topic>${namespace}/scan</topic>
+                <gz_frame_id>${lidar_name}_frame</gz_frame_id>
             </sensor>
         </gazebo>
