Commit message: added oak d macro

File: src/microros_hardware_interface/description/urdf/core.urdf.xacro (robot description, xacro)
@@ -12,4 +12,5 @@
   <xacro:include filename="$(find microros_hardware_interface)/description/urdf/util/macros/imu.xacro" />
   <xacro:include filename="$(find microros_hardware_interface)/description/urdf/util/macros/lidar.xacro" />
+  <xacro:include filename="$(find microros_hardware_interface)/description/urdf/util/macros/oakd.xacro" />
   <!-- Import Robot Description -->
   <xacro:include filename="$(find microros_hardware_interface)/description/urdf/robot.urdf.xacro" />
@@ -20,17 +21,10 @@
   <xacro:robot_hardware prefix="$(arg prefix)" />
   <xacro:micro_system_hardware_ros2_control name="MicroSystemHardware" prefix="$(arg prefix)"/>
-  <!-- Import Camera -->
-  <!-- <xacro:include filename="$(find microros_hardware_interface)/description/urdf/util/components/camera.xacro" /> -->
-  <!-- <xacro:camera prefix="$(arg prefix)"/> -->
-  <xacro:include filename="$(find microros_hardware_interface)/description/urdf/util/components/driver_camera.xacro" />
-  <!-- Import Depth Camera -->
-  <!-- <xacro:include filename="$(find microros_hardware_interface)/description/urdf/util/components/depth_camera.xacro" /> -->
-  <!-- <xacro:depth_camera prefix="$(arg prefix)"/> -->
-  <xacro:camera cam_name="rgbd_camera" namespace="rgbd_camera" parent="chassis_link" x="0.1" y="0" z="0.1" roll="0" pitch="0" yaw="0"/>
-  <!-- Import LiDAR -->
-  <!-- <xacro:include filename="$(find microros_hardware_interface)/description/urdf/util/components/lidar.xacro" />
-  <xacro:lidar prefix="$(arg prefix)"/> -->
-  <xacro:lidar lidar_name="laser" namespace="lidar" parent="chassis_link" x="0" y="0" z="0.14" roll="0" pitch="0" yaw="0"/>
-  <!-- Create IMU -->
-  <xacro:imu imu_name="imu" namespace="imu" parent="chassis_link" x="0.1" y="0" z="0.17" roll="0" pitch="0" yaw="0"/>
+  <!-- Hardware Components -->
+    <!-- Import Driver Camera -->
+    <xacro:include filename="$(find microros_hardware_interface)/description/urdf/util/components/driver_camera.xacro" />
+    <!-- Import OakD -->
+    <xacro:include filename="$(find microros_hardware_interface)/description/urdf/util/components/front_oakd.xacro" />
+    <!-- Import LiDAR -->
+    <xacro:include filename="$(find microros_hardware_interface)/description/urdf/util/components/rplidar.xacro" />
 </robot>

File: src/microros_hardware_interface/description/urdf/util/components/driver_camera.xacro (robot description, xacro)
@@ -1,4 +1,4 @@
 <?xml version="1.0"?>
 <robot xmlns:xacro="http://www.ros.org/wiki/xacro" >
-    <xacro:camera cam_name="camera" namespace="camera" parent="chassis_link" x="0" y="0" z="${base_height}" roll="0" pitch="0" yaw="0"/>
+    <xacro:camera name="camera" namespace="camera" parent="chassis_link" x="0" y="0" z="${base_height}" roll="0" pitch="0" yaw="0"/>
 </robot>

File: src/microros_hardware_interface/description/urdf/util/macros/camera.xacro (robot description, xacro)
@@ -1,8 +1,8 @@
 <?xml version="1.0"?>
 <robot xmlns:xacro="http://www.ros.org/wiki/xacro" >
-    <xacro:macro name="camera" params="cam_name namespace parent x:=0 y:=0 z:=0 roll:=0 pitch:=0 yaw:=0">
+    <xacro:macro name="camera" params="name namespace parent x:=0 y:=0 z:=0 roll:=0 pitch:=0 yaw:=0">
         <xacro:property name="PI" value="3.1415926535897931"/>
         <!-- main link -->
-        <link name="${cam_name}_link">
+        <link name="${name}_link">
             <visual>
                 <geometry>
@@ -13,19 +13,19 @@
         </link>
         <!-- optical link -->
-        <link name="${cam_name}_link_optical"></link>
+        <link name="${name}_link_optical"></link>
         <!-- main joint -->
-        <joint name="${cam_name}_joint" type="fixed">
+        <joint name="${name}_joint" type="fixed">
             <parent link="${parent}"/>
-            <child link="${cam_name}_link"/>
+            <child link="${name}_link"/>
             <origin xyz="${x} ${y} ${z}" rpy="${roll} ${pitch} ${yaw}"/>
         </joint>
         <!-- optical joint -->
-        <joint name="${cam_name}_optical_joint" type="fixed">
-            <parent link="${cam_name}_link"/>
-            <child link="${cam_name}_link_optical"/>
+        <joint name="${name}_optical_joint" type="fixed">
+            <parent link="${name}_link"/>
+            <child link="${name}_link_optical"/>
             <origin xyz="0 0 0" rpy="${-PI / 2} 0 ${-PI / 2}"/>
         </joint>
         <!-- gazebo reference -->
-        <gazebo reference="${cam_name}_link">
+        <gazebo reference="${name}_link">
             <material>Gazebo/Black</material>
             <sensor name="${namespace}" type="camera">
@@ -50,5 +50,5 @@
                 </camera>
                 <topic>${namespace}/image_raw</topic>
-                <gz_frame_id>${cam_name}_link_optical</gz_frame_id>
+                <gz_frame_id>${name}_link_optical</gz_frame_id>
             </sensor>
         </gazebo>

File: src/microros_hardware_interface/description/urdf/util/macros/depth_camera.xacro (robot description, xacro)
@@ -1,8 +1,8 @@
 <?xml version="1.0"?>
 <robot xmlns:xacro="http://www.ros.org/wiki/xacro" >
-    <xacro:macro name="depth_camera" params="cam_name namespace parent x:=0 y:=0 z:=0 roll:=0 pitch:=0 yaw:=0">
+    <xacro:macro name="depth_camera" params="name namespace parent x:=0 y:=0 z:=0 roll:=0 pitch:=0 yaw:=0">
         <xacro:property name="PI" value="3.1415926535897931"/>
         <!-- main link -->
-        <link name="${cam_name}_link">
+        <link name="${name}_link">
             <visual>
                 <geometry>
@@ -13,18 +13,18 @@
         </link>
         <!-- optical link -->
-        <link name="${cam_name}_link_optical"></link>
+        <link name="${name}_link_optical"></link>
         <!-- main joint -->
-        <joint name="${cam_name}_joint" type="fixed">
+        <joint name="${name}_joint" type="fixed">
             <parent link="${parent}"/>
-            <child link="${cam_name}_link"/>
+            <child link="${name}_link"/>
             <origin xyz="${x} ${y} ${z}" rpy="${roll} ${pitch} ${yaw}"/>
         </joint>
         <!-- optical joint -->
-        <joint name="${cam_name}_optical_joint" type="fixed">
-            <parent link="${cam_name}_link"/>
-            <child link="${cam_name}_link_optical"/>
+        <joint name="${name}_optical_joint" type="fixed">
+            <parent link="${name}_link"/>
+            <child link="${name}_link_optical"/>
             <origin xyz="0 0 0" rpy="${-PI / 2} 0 ${-PI / 2}"/>
         </joint>
-        <gazebo reference="${cam_name}_link">
+        <gazebo reference="${name}_link">
             <material>Gazebo/Black</material>
             <sensor name="${namespace}" type="rgbd_camera">
@@ -55,5 +55,5 @@
                 </camera>
                 <topic>${namespace}</topic>
-                <gz_frame_id>${cam_name}_link_optical</gz_frame_id>
+                <gz_frame_id>${name}_link_optical</gz_frame_id>
                 <!-- <plugin filename="RosGzPointCloud" name="ros_gz_point_cloud::PointCloud">
                     <namespace>rgbd_camera</namespace>

File: src/microros_hardware_interface/description/urdf/util/macros/imu.xacro (robot description, xacro)
@@ -1,7 +1,7 @@
 <?xml version="1.0"?>
 <robot xmlns:xacro="http://www.ros.org/wiki/xacro" >
-    <xacro:macro name="imu" params="imu_name namespace parent x:=0 y:=0 z:=0 roll:=0 pitch:=0 yaw:=0">
+    <xacro:macro name="imu" params="name namespace parent x:=0 y:=0 z:=0 roll:=0 pitch:=0 yaw:=0">
         <xacro:property name="PI" value="3.1415926535897931"/>
-        <link name="${imu_name}_link">
+        <link name="${name}_link">
             <visual>
                 <geometry>
@@ -11,12 +11,12 @@
             </visual>
         </link>
-        <joint name="${imu_name}_joint" type="fixed">
+        <joint name="${name}_joint" type="fixed">
             <parent link="${parent}"/>
-            <child link="${imu_name}_link"/>
+            <child link="${name}_link"/>
             <origin xyz="${x} ${y} ${z}" rpy="${roll} ${pitch} ${yaw}"/>
         </joint>
-        <gazebo reference="${imu_name}_link">
+        <gazebo reference="${name}_link">
             <material>Gazebo/Black</material>
-            <sensor name="${imu_name}" type="imu">
+            <sensor name="${name}" type="imu">
                 <!-- offset from joint -->
                 <pose> 0 0 0 0 0 0 </pose>
@@ -28,5 +28,5 @@
                 <update_rate>30</update_rate>
                 <topic>${namespace}/data</topic>
-                <gz_frame_id>${imu_name}_link</gz_frame_id>
+                <gz_frame_id>${name}_link</gz_frame_id>
                 <plugin filename="gz-sim-imu-system" name="gz::sim::systems::Imu"/>
             </sensor>

File: src/microros_hardware_interface/description/urdf/util/macros/lidar.xacro (robot description, xacro)
@@ -1,11 +1,11 @@
 <?xml version="1.0"?>
 <robot xmlns:xacro="http://www.ros.org/wiki/xacro" >
-    <xacro:macro name="lidar" params="lidar_name namespace parent x:=0 y:=0 z:=0 roll:=0 pitch:=0 yaw:=0">
-        <joint name="${lidar_name}_joint" type="fixed">
+    <xacro:macro name="lidar" params="name namespace parent x:=0 y:=0 z:=0 roll:=0 pitch:=0 yaw:=0">
+        <joint name="${name}_joint" type="fixed">
             <parent link="${parent}"/>
-            <child link="${lidar_name}_frame"/>
+            <child link="${name}_frame"/>
             <origin xyz="${x} ${y} ${z}" rpy="${roll} ${pitch} ${yaw}"/>
         </joint>
-        <link name="${lidar_name}_frame">
+        <link name="${name}_frame">
             <visual>
                 <geometry>
@@ -15,7 +15,7 @@
             </visual>
         </link>
-        <gazebo reference="${lidar_name}_frame">
+        <gazebo reference="${name}_frame">
             <material>Gazebo/Blue</material>
-            <sensor name="${lidar_name}" type="gpu_lidar">
+            <sensor name="${name}" type="gpu_lidar">
                 <pose> 0 0 0 0 0 0 </pose>
                 <visualize>true</visualize>
@@ -35,5 +35,5 @@
                 </lidar>
                 <topic>${namespace}/scan</topic>
-                <gz_frame_id>${lidar_name}_frame</gz_frame_id>
+                <gz_frame_id>${name}_frame</gz_frame_id>
             </sensor>
         </gazebo>

Commit message: used actual coordinates for oak d and added visualize param for components

File: src/microros_hardware_interface/description/urdf/core.urdf.xacro (robot description, xacro)
@@ -24,5 +24,5 @@
     <!-- Import Driver Camera -->
     <xacro:include filename="$(find microros_hardware_interface)/description/urdf/util/components/driver_camera.xacro" />
-    <!-- Import OakD -->
+    <!-- Import Oak-D -->
     <xacro:include filename="$(find microros_hardware_interface)/description/urdf/util/components/front_oakd.xacro" />
     <!-- Import LiDAR -->

File: src/microros_hardware_interface/description/urdf/util/components/front_oakd.xacro (robot description, xacro)
@@ -1,4 +1,4 @@
 <?xml version="1.0"?>
 <robot xmlns:xacro="http://www.ros.org/wiki/xacro" >
-    <xacro:oakd name="oakd" namespace="oak" parent="chassis_link" x="0.5" y="0" z="${base_height}" roll="0" pitch="0" yaw="0"/>
+    <xacro:oakd name="oakd" namespace="oak" parent="chassis_link" x="0.15" y="0" z="0.2" roll="0" pitch="0" yaw="0"/>
 </robot>

File: src/microros_hardware_interface/description/urdf/util/macros/camera.xacro (robot description, xacro)
@@ -1,5 +1,5 @@
 <?xml version="1.0"?>
 <robot xmlns:xacro="http://www.ros.org/wiki/xacro" >
-    <xacro:macro name="camera" params="name namespace parent x:=0 y:=0 z:=0 roll:=0 pitch:=0 yaw:=0">
+    <xacro:macro name="camera" params="name namespace parent x:=0 y:=0 z:=0 roll:=0 pitch:=0 yaw:=0 visualize:=true">
         <xacro:property name="PI" value="3.1415926535897931"/>
         <!-- main link -->
@@ -7,5 +7,7 @@
             <visual>
                 <geometry>
-                    <box size="0.010 0.03 0.03"/>
+                    <xacro:if value="${visualize}">
+                        <box size="0.010 0.03 0.03"/>
+                    </xacro:if>
                 </geometry>
                 <material name="black"/>

File: src/microros_hardware_interface/description/urdf/util/macros/depth_camera.xacro (robot description, xacro)
@@ -1,5 +1,5 @@
 <?xml version="1.0"?>
 <robot xmlns:xacro="http://www.ros.org/wiki/xacro" >
-    <xacro:macro name="depth_camera" params="name namespace parent x:=0 y:=0 z:=0 roll:=0 pitch:=0 yaw:=0">
+    <xacro:macro name="depth_camera" params="name namespace parent x:=0 y:=0 z:=0 roll:=0 pitch:=0 yaw:=0 visualize:=true">
         <xacro:property name="PI" value="3.1415926535897931"/>
         <!-- main link -->
@@ -7,5 +7,7 @@
             <visual>
                 <geometry>
-                    <box size="0.010 0.03 0.03"/>
+                    <xacro:if value="${visualize}">
+                        <box size="0.010 0.03 0.03"/>
+                    </xacro:if>
                 </geometry>
                 <material name="black"/>

File: src/microros_hardware_interface/description/urdf/util/macros/imu.xacro (robot description, xacro)
@@ -1,10 +1,12 @@
 <?xml version="1.0"?>
 <robot xmlns:xacro="http://www.ros.org/wiki/xacro" >
-    <xacro:macro name="imu" params="name namespace parent x:=0 y:=0 z:=0 roll:=0 pitch:=0 yaw:=0">
+    <xacro:macro name="imu" params="name namespace parent x:=0 y:=0 z:=0 roll:=0 pitch:=0 yaw:=0 visualize:=true">
         <xacro:property name="PI" value="3.1415926535897931"/>
         <link name="${name}_link">
             <visual>
                 <geometry>
-                    <box size="0.010 0.03 0.03"/>
+                    <xacro:if value="${visualize}">
+                        <box size="0.010 0.03 0.03"/>
+                    </xacro:if>
                 </geometry>
                 <material name="black"/>

File: src/microros_hardware_interface/description/urdf/util/macros/lidar.xacro (robot description, xacro)
@@ -1,5 +1,5 @@
 <?xml version="1.0"?>
 <robot xmlns:xacro="http://www.ros.org/wiki/xacro" >
-    <xacro:macro name="lidar" params="name namespace parent x:=0 y:=0 z:=0 roll:=0 pitch:=0 yaw:=0">
+    <xacro:macro name="lidar" params="name namespace parent x:=0 y:=0 z:=0 roll:=0 pitch:=0 yaw:=0 visualize:=true">
         <joint name="${name}_joint" type="fixed">
             <parent link="${parent}"/>
@@ -10,5 +10,7 @@
             <visual>
                 <geometry>
-                    <cylinder radius="0.05" length="0.04"/>
+                    <xacro:if value="${visualize}">
+                        <cylinder radius="0.05" length="0.04"/>
+                    </xacro:if>
                 </geometry>
                 <material name="blue"/>

File: src/microros_hardware_interface/description/urdf/util/macros/oakd.xacro (robot description, xacro)
@@ -2,22 +2,28 @@
 <robot xmlns:xacro="http://www.ros.org/wiki/xacro" >
     <xacro:macro name="oakd" params="name namespace parent x:=0 y:=0 z:=0 roll:=0 pitch:=0 yaw:=0">
-        <link name="${name}_base_link">
+        <link name="${name}-base-frame"/>
+        <link name="${name}">
             <visual>
+                <origin xyz="0 0 0" rpy="${PI / 2} 0 ${PI / 2}"/>
                 <geometry>
-                     <box size="0.010 0.03 0.03"/>
-                    <!-- <mesh filename="file://$(find microros_hardware_interface)/description/urdf/assets/components/oakd.STL"/> -->
+                    <mesh filename="file://$(find microros_hardware_interface)/description/urdf/assets/components/Oak-D.stl"/>
                 </geometry>
-                <material name="black"/>
+                <!-- <material name="black"/> -->
             </visual>
         </link>
-        <joint name="${name}_base_joint" type="fixed">
+        <joint name="${name}_joint" type="fixed">
+            <parent link="${name}-base-frame"/>
+            <child link="${name}"/>
+            <origin xyz="0 0 0" rpy="0 0 0"/>
+        </joint>
+        <joint name="${name}-base-frame_joint" type="fixed">
             <parent link="${parent}"/>
-            <child link="${name}_base_link"/>
+            <child link="${name}-base-frame"/>
             <origin xyz="${x} ${y} ${z}" rpy="${roll} ${pitch} ${yaw}"/>
         </joint>
-        <xacro:depth_camera name="${name}_depth" namespace="${namespace}/depth" parent="${name}_base_link" x="0" y="0" z="0" roll="0" pitch="0" yaw="0"/>
-        <xacro:camera name="${name}_left" namespace="${namespace}/left" parent="${name}_base_link" x="0" y="0.05" z="0" roll="0" pitch="0" yaw="0"/>
-        <xacro:camera name="${name}_right" namespace="${namespace}/right" parent="${name}_base_link" x="0" y="-0.05" z="0" roll="0" pitch="0" yaw="0"/>
-        <xacro:imu name="${name}_imu" namespace="${namespace}/imu" parent="${name}_base_link" x="0" y="0" z="0" roll="0" pitch="0" yaw="0"/>
+        <xacro:depth_camera name="${name}_rgb" namespace="${namespace}/rgb" parent="${name}" x="0.0073" y="0" z="0" roll="0" pitch="0" yaw="0" visualize="false"/>
+        <xacro:camera name="${name}_left" namespace="${namespace}/left" parent="${name}" x="0.0073" y="0.0375" z="0" roll="0" pitch="0" yaw="0" visualize="false"/>
+        <xacro:camera name="${name}_right" namespace="${namespace}/right" parent="${name}" x="0.0073" y="-0.0375" z="0" roll="0" pitch="0" yaw="0" visualize="false"/>
+        <xacro:imu name="${name}_imu" namespace="${namespace}/imu" parent="${name}" x="0" y="0" z="0" roll="0" pitch="0" yaw="0" visualize="false"/>
     </xacro:macro>
 </robot>
