Commit message: added depth camera and imu to simulation

File: src/microros_hardware_interface/description/urdf/components/depth_camera.xacro (robot description, xacro)
@@ -1,18 +1,18 @@
 <?xml version="1.0"?>
 <robot xmlns:xacro="http://www.ros.org/wiki/xacro" >
-    <xacro:macro name="camera" params="prefix">
+    <xacro:macro name="depth_camera" params="prefix">
         <xacro:property name="x_transform" value="0.1778"/>
         <xacro:property name="y_transform" value="0"/>
-        <xacro:property name="z_transform" value="0.03"/>
+        <xacro:property name="z_transform" value="0.1"/>
         <xacro:property name="r_transform" value="0"/>
         <xacro:property name="p_transform" value="0"/>
         <xacro:property name="y_transform" value="0"/>
         <xacro:property name="PI" value="3.1415926535897931"/>
-        <joint name="${prefix}camera_joint" type="fixed">
+        <joint name="${prefix}depth_camera_joint" type="fixed">
             <parent link="${prefix}chassis_link"/>
-            <child link="${prefix}camera_link"/>
+            <child link="${prefix}depth_camera_link"/>
             <origin xyz="${x_transform / 2} ${y_transform} ${z_transform}" rpy="${r_transform} ${p_transform} ${y_transform}"/>
         </joint>
-        <link name="${prefix}camera_link">
+        <link name="${prefix}depth_camera_link">
             <visual>
                 <geometry>
@@ -22,15 +22,16 @@
             </visual>
         </link>
-        <joint name="${prefix}camera_optical_joint" type="fixed">
-            <parent link="${prefix}camera_link"/>
-            <child link="${prefix}camera_link_optical"/>
+        <joint name="${prefix}depth_camera_optical_joint" type="fixed">
+            <parent link="${prefix}depth_camera_link"/>
+            <child link="${prefix}depth_camera_link_optical"/>
             <origin xyz="${x_transform / 2} ${y_transform} ${z_transform}" rpy="${-PI / 2} 0 ${-PI / 2}"/>
         </joint>
-        <link name="${prefix}camera_link_optical"></link>
-        <gazebo reference="${prefix}camera_link">
+        <link name="${prefix}depth_camera_link_optical"></link>
+        <gazebo reference="${prefix}depth_camera_link">
             <material>Gazebo/Black</material>
-            <sensor name="camera" type="depth">
+            <sensor name="rgbd_camera" type="rgbd_camera">
                 <pose> 0 0 0 0 0 0 </pose>
                 <visualize>true</visualize>
+                <always_on>1</always_on>
                 <update_rate>30</update_rate>
                 <camera>
@@ -43,12 +44,19 @@
                     <clip>
                         <near>0.05</near>
-                        <far>8.0</far>
+                        <far>8</far>
                     </clip>
+                    <noise>
+						<type>gaussian</type>
+						<mean>0.0</mean>
+						<stddev>0.01</stddev>
+					</noise>
                 </camera>
-                <plugin name="camera_controller" filename="libgazebo_ros_camera.so">
-                    <frame_name>camera_link_optical</frame_name>
-                    <min_depth>0.1</min_depth>
-                    <max_depth>100.0</max_depth>
-                </plugin>
+                <topic>rgbd_camera</topic>
+                <gz_frame_id>depth_camera_link_optical</gz_frame_id>
+                <!-- <plugin filename="RosGzPointCloud" name="ros_gz_point_cloud::PointCloud">
+                    <namespace>rgbd_camera</namespace>
+                    <topic>points</topic>
+                    <frame_id>camera_link_optical</frame_id>
+                </plugin> -->
             </sensor>
         </gazebo>

File: src/microros_hardware_interface/description/urdf/core.urdf.xacro (robot description, xacro)
@@ -14,12 +14,15 @@
   <xacro:robot_hardware prefix="$(arg prefix)" />
   <xacro:micro_system_hardware_ros2_control name="MicroSystemHardware" prefix="$(arg prefix)" />
-  <!-- <xacro:include filename="$(find microros_hardware_interface)/ros2_control/sim.xacro"/> -->
   <!-- Import Camera -->
   <xacro:include filename="$(find microros_hardware_interface)/description/urdf/components/camera.xacro" />
   <xacro:camera prefix="$(arg prefix)"/>
   <!-- Import Depth Camera -->
-  <!-- <xacro:include filename="$(find microros_hardware_interface)/urdf/components/depth_camera.xacro" /> -->
+  <xacro:include filename="$(find microros_hardware_interface)/description/urdf/components/depth_camera.xacro" />
+  <xacro:depth_camera prefix="$(arg prefix)"/>
   <!-- Import LiDAR -->
   <xacro:include filename="$(find microros_hardware_interface)/description/urdf/components/lidar.xacro" />
   <xacro:lidar prefix="$(arg prefix)"/>
+  <!-- Import IMU -->
+  <xacro:include filename="$(find microros_hardware_interface)/description/urdf/components/imu.xacro" />
+  <xacro:imu prefix="$(arg prefix)"/>
 </robot>
