Commit message: fixed visualize to eliminate empty children

File: src/microros_hardware_interface/description/urdf/util/macros/camera.xacro (robot description, xacro)
@@ -5,12 +5,12 @@
         <!-- main link -->
         <link name="${name}_link">
-            <visual>
-                <geometry>
-                    <xacro:if value="${visualize}">
-                        <box size="0.010 0.03 0.03"/>
-                    </xacro:if>
-                </geometry>
-                <material name="black"/>
-            </visual>
+            <xacro:if value="${visualize}">
+                <visual>
+                    <geometry>
+                            <box size="0.010 0.03 0.03"/>
+                    </geometry>
+                    <material name="black"/>
+                </visual>
+            </xacro:if>
         </link>
         <!-- optical link -->

File: src/microros_hardware_interface/description/urdf/util/macros/depth_camera.xacro (robot description, xacro)
@@ -5,12 +5,12 @@
         <!-- main link -->
         <link name="${name}_link">
-            <visual>
-                <geometry>
-                    <xacro:if value="${visualize}">
+             <xacro:if value="${visualize}">
+                <visual>
+                    <geometry>
                         <box size="0.010 0.03 0.03"/>
-                    </xacro:if>
-                </geometry>
-                <material name="black"/>
-            </visual>
+                    </geometry>
+                    <material name="black"/>
+                </visual>
+            </xacro:if>
         </link>
         <!-- optical link -->

File: src/microros_hardware_interface/description/urdf/util/macros/imu.xacro (robot description, xacro)
@@ -4,12 +4,12 @@
         <xacro:property name="PI" value="3.1415926535897931"/>
         <link name="${name}_link">
-            <visual>
-                <geometry>
-                    <xacro:if value="${visualize}">
-                        <box size="0.010 0.03 0.03"/>
-                    </xacro:if>
-                </geometry>
-                <material name="black"/>
-            </visual>
+            <xacro:if value="${visualize}">
+                <visual>
+                    <geometry>
+                            <box size="0.010 0.03 0.03"/>
+                    </geometry>
+                    <material name="black"/>
+                </visual>
+            </xacro:if>
         </link>
         <joint name="${name}_joint" type="fixed">

File: src/microros_hardware_interface/description/urdf/util/macros/lidar.xacro (robot description, xacro)
@@ -8,12 +8,12 @@
         </joint>
         <link name="${name}_frame">
-            <visual>
-                <geometry>
-                    <xacro:if value="${visualize}">
+            <xacro:if value="${visualize}">
+                <visual>
+                    <geometry>
                         <cylinder radius="0.05" length="0.04"/>
-                    </xacro:if>
-                </geometry>
-                <material name="blue"/>
-            </visual>
+                    </geometry>
+                    <material name="blue"/>
+                </visual>
+            </xacro:if>
         </link>
         <gazebo reference="${name}_frame">
