Commit message: fixed caster wheel not being proper size for collision

File: src/microros_hardware_interface/description/urdf/util/macros/dead_wheel.xacro (robot description, xacro)
@@ -8,5 +8,5 @@
                 <geometry>
                     <!-- <mesh filename="file://$(find microros_hardware_interface)/description/urdf/assets/wheel/Wheel.stl"/> -->
-                    <sphere radius="${wheel_radius}" />
+                    <sphere radius="0.04800000" />
                 </geometry>
                 <!-- <surface>
