Commit message: fixed urdf to match the model

File: src/microros_hardware_interface/description/urdf/util/constants.xacro (robot description, xacro)
@@ -2,5 +2,5 @@
 <robot xmlns:xacro="http://www.ros.org/wiki/xacro">
     <xacro:property name="PI" value="3.1415926535897931"/>
-    <xacro:property name="base_mass" value="1" /> <!-- arbitrary value for base mass -->
+    <xacro:property name="base_mass" value="4" /> <!-- arbitrary value for base mass -->
     <xacro:property name="base_width" value="0.240" />
     <xacro:property name="base_length" value="0.300" />
@@ -10,5 +10,5 @@
     <xacro:property name="wheel_radius" value="0.032" />
     <xacro:property name="wheel_mass" value="0.34055" /> <!-- arbitrary value for wheel mass -->
-    <xacro:property name="friction" value="1"/>
+    <xacro:property name="friction" value="10"/>
     <xacro:property name="min_depth" value="0.5"/>
     <xacro:property name="damping" value="0.001"/>

File: src/microros_hardware_interface/description/urdf/util/macros/dead_wheel.xacro (robot description, xacro)
@@ -29,8 +29,8 @@
             <!-- VISIUAL -->
             <visual>
-                <origin xyz="0 0 0" rpy="${side * -PI/2} 0 0"/>
+                <origin xyz="0 0 0" rpy="0 0 0"/>
                 <geometry>
-                    <mesh filename="file://$(find microros_hardware_interface)/description/urdf/assets/wheel/Wheel.obj"/>
-                    <!-- <sphere radius="${wheel_radius}" /> -->
+                    <mesh filename="file://$(find microros_hardware_interface)/description/urdf/assets/caster/caster.obj"/>
+                    <!-- <sphere radius="${wheel_radius / 5}" /> -->
                 </geometry>
                 <!-- <material name="black"/> -->
@@ -54,5 +54,5 @@
             <parent link="${prefix}chassis_link"/>
             <child link="${name}_wheel"/>
-            <origin xyz="${front * .120} ${side * .129} -.0199" rpy="0 0 0"/>
+            <origin xyz="${front * 0.10855000} ${side * 0.08160000} -0.01194906" rpy="0 0 0"/>
         </joint>
     </xacro:macro>

File: src/microros_hardware_interface/description/urdf/util/macros/wheel.xacro (robot description, xacro)
@@ -53,6 +53,6 @@
         <gazebo reference="${name}_wheel">
             <material>Gazebo/Black</material>
-            <mu1 value="1"/>
-            <mu2 value="1"/>
+            <mu1 value="10"/>
+            <mu2 value="10"/>
         </gazebo>
         <joint name="${name}_wheel_joint" type="continuous">
@@ -60,5 +60,5 @@
             <child link="${name}_wheel"/>
             <origin xyz="${front * .120} ${side * .129} -.0199" rpy="0 0 0"/>
-            <axis xyz="0 1 0"/>
+            <axis xyz="0 -1 0"/>
             <limit effort="1000.0" velocity="100.0"/>
             <dynamics damping="${damping}"/>
