Commit message: changed coordinates for wheels

File: ros2_ws/src/microros_hardware_interface/description/urdf/util/components/front_oakd.xacro (robot description, xacro)
@@ -1,4 +1,4 @@
 <?xml version="1.0"?>
 <robot xmlns:xacro="http://www.ros.org/wiki/xacro" >
-    <xacro:oakd name="oakd" namespace="oak" parent="chassis_link" x="0.15" y="0" z="0.2" roll="0" pitch="0" yaw="0"/>
+    <xacro:oakd name="oakd" namespace="oak" parent="chassis_link" x="-0.15" y="0" z="0.2" roll="0" pitch="0" yaw="${PI}"/>
 </robot>

File: ros2_ws/src/microros_hardware_interface/description/urdf/util/macros/wheel.xacro (robot description, xacro)
@@ -5,5 +5,5 @@
             <!-- COLLISION -->
             <collision>
-            <origin xyz="0 0 0" rpy="${side * -PI/2} 0 0"/>
+            <origin xyz="0 0 0" rpy="0 0 0"/>
             <geometry>
                 <!-- <mesh filename="file://$(find microros_hardware_interface)/description/urdf/assets/wheel/Wheel.stl"/> -->
@@ -34,5 +34,5 @@
             <!-- VISIUAL -->
             <visual>
-                <origin xyz="0 0 0" rpy="${side * -PI/2} 0 0"/>
+                <origin xyz="0 0 0" rpy="0 0 0"/>
                 <geometry>
                     <mesh filename="file://$(find microros_hardware_interface)/description/urdf/assets/wheel/Wheel.obj"/>
@@ -59,6 +59,6 @@
             <parent link="${prefix}chassis_link"/>
             <child link="${name}_wheel"/>
-            <origin xyz="${front * .120} ${side * .129} -.0199" rpy="0 0 0"/>
-            <axis xyz="0 -1 0"/>
+            <origin xyz="${front * .120} ${side * .129} -.0199" rpy="${side * -PI/2}  0 0"/>
+            <axis xyz="0 0 ${side}"/>
             <limit effort="1000.0" velocity="100.0"/>
             <dynamics damping="${damping}"/>
