Commit message: fixed transforms

File: ros2_ws/src/microros_hardware_interface/description/urdf/robot.urdf.xacro (robot description, xacro)
@@ -35,5 +35,5 @@
       <parent link="${prefix}base_link"/>
       <child link="${prefix}chassis_link"/>
-      <origin xyz="0 0 ${.0199 + wheel_radius}" rpy="0 0 0"/>
+      <origin xyz="0 0 ${.0199 + wheel_radius}" rpy="0 0 ${PI}"/>
       <axis xyz="0 0 1"/>
       <dynamics damping="${damping}"/>

File: ros2_ws/src/microros_hardware_interface/description/urdf/util/macros/wheel.xacro (robot description, xacro)
@@ -60,5 +60,5 @@
             <child link="${name}_wheel"/>
             <origin xyz="${front * .120} ${side * .129} -.0199" rpy="${side * -PI/2}  0 0"/>
-            <axis xyz="0 0 ${side}"/>
+            <axis xyz="0 0 ${-side}"/>
             <limit effort="1000.0" velocity="100.0"/>
             <dynamics damping="${damping}"/>

Commit message: added slam toolbox

File: ros2_ws/src/microros_hardware_interface/description/urdf/robot.urdf.xacro (robot description, xacro)
@@ -4,4 +4,6 @@
     <!-- Base Link -->
     <link name="${prefix}base_link"/>
+    <!-- Base Footprint -->
+    <link name="${prefix}base_footprint"/>
     <!-- Chassis -->
     <link name="${prefix}chassis_link">
@@ -39,4 +41,9 @@
       <dynamics damping="${damping}"/>
     </joint>
+    <joint name="${prefix}base_footprint_joint" type="fixed">
+      <parent link="${prefix}base_link"/>
+      <child link="${prefix}base_footprint"/>
+      <origin xyz="0 0 0" rpy="0 0 0"/>
+    </joint>
     <!--front is positive, left is positive-->
     <xacro:wheel name="left" x="0" y="0" z="0" front="-1" side="-1"/>

File: ros2_ws/src/microros_hardware_interface/description/urdf/util/macros/dead_wheel.xacro (robot description, xacro)
@@ -8,5 +8,5 @@
                 <geometry>
                     <!-- <mesh filename="file://$(find microros_hardware_interface)/description/urdf/assets/wheel/Wheel.stl"/> -->
-                    <sphere radius="0.04800000" />
+                    <sphere radius="0.03605094" />
                 </geometry>
                 <!-- <surface>
@@ -31,6 +31,6 @@
                 <origin xyz="0 0 0" rpy="0 0 0"/>
                 <geometry>
-                    <mesh filename="file://$(find microros_hardware_interface)/description/urdf/assets/caster/caster.obj"/>
-                    <!-- <sphere radius="${wheel_radius / 5}" /> -->
+                    <!-- <mesh filename="file://$(find microros_hardware_interface)/description/urdf/assets/caster/caster.obj"/> -->
+                    <sphere radius="0.03605094" />
                 </geometry>
                 <!-- <material name="black"/> -->

File: ros2_ws/src/microros_hardware_interface/description/urdf/util/macros/lidar.xacro (robot description, xacro)
@@ -33,5 +33,5 @@
                     <range>
                         <min>0.3</min>
-                        <max>12</max>
+                        <max>20</max>
                     </range>
                 </lidar>
