Commit message: added slam_toolbox

File: ros2_ws/src/microros_hardware_interface/description/urdf/util/macros/dead_wheel.xacro (robot description, xacro)
@@ -31,6 +31,6 @@
                 <origin xyz="0 0 0" rpy="0 0 0"/>
                 <geometry>
-                    <!-- <mesh filename="file://$(find microros_hardware_interface)/description/urdf/assets/caster/caster.obj"/> -->
-                    <sphere radius="0.03605094" />
+                    <mesh filename="file://$(find microros_hardware_interface)/description/urdf/assets/caster/caster.obj"/>
+                    <!-- <sphere radius="0.03605094" /> -->
                 </geometry>
                 <!-- <material name="black"/> -->

File: ros2_ws/src/microros_hardware_interface/description/urdf/util/macros/wheel.xacro (robot description, xacro)
@@ -59,5 +59,5 @@
             <parent link="${prefix}chassis_link"/>
             <child link="${name}_wheel"/>
-            <origin xyz="${front * .120} ${side * .129} -.0199" rpy="${side * -PI/2}  0 0"/>
+            <origin xyz="${front * .120} ${side * .129} -0.016" rpy="${side * -PI/2}  0 0"/>
             <axis xyz="0 0 ${-side}"/>
             <limit effort="1000.0" velocity="100.0"/>
