Commit message: Working version of hardware

File: ros2_ws/src/robot_hardware/description/ros2_control/robot_hardware.ros2_control.xacro (robot description, xacro)
@@ -3,25 +3,9 @@
 <xacro:macro name="robot_hardware_ros2_control" params="name prefix">
     <xacro:property name="speed_multiplier" value="1"/>
-    <xacro:macro name="front_wheel" params="name">
+    <xacro:macro name="wheel" params="name">
         <joint name="${name}_wheel_joint">
             <command_interface name="velocity"/>
-            <!-- RC car doesn't have feedback -->
-            <!-- <state_interface name="velocity"/> -->
-            <!-- <state_interface name="position"/> -->
-            <!-- <state_interface name="effort"/> -->
-        </joint>
-        <joint name="${name}_steer_joint">
-            <command_interface name="position"/>
-            <!-- <state_interface name="position"/> -->
-            <state_interface name="effort"/>
-        </joint>
-    </xacro:macro>
-    <xacro:macro name="rear_wheel" params="name">
-        <joint name="${name}_wheel_joint">
-            <command_interface name="velocity"/>
-            <!-- RC car doesn't have feedback -->
-            <!-- <state_interface name="velocity"/> -->
+            <state_interface name="velocity"/>
             <state_interface name="position"/>
-            <!-- <state_interface name="effort"/> -->
         </joint>
     </xacro:macro>
@@ -34,11 +18,7 @@
                 <param name="MCU_field">product</param>
                 <param name="MCU_description">STM32 Virtual ComPort</param>
-                <!-- <param name="my_int_param">0</param> -->
-                <!-- <param name="my_string_param">Hello World</param> -->
             </hardware>
-            <xacro:front_wheel name="${prefix}front_left"/>
-            <xacro:front_wheel name="${prefix}front_right"/>
-            <xacro:rear_wheel name="${prefix}rear_left"/>
-            <xacro:rear_wheel name="${prefix}rear_right"/>
+            <xacro:wheel name="${prefix}left"/>
+            <xacro:wheel name="${prefix}right"/>
         </ros2_control>
     </xacro:unless>
@@ -50,104 +30,29 @@
             <plugin>gz_ros2_control/GazeboSimSystem</plugin>
             </hardware>
-            <!-- drive joint -->
-            <joint name="${prefix}virtual_rear_wheel_joint">
-            <command_interface name="velocity">
-                <param name="min">-1000</param>
-                <param name="max">1000</param>
-            </command_interface>
-            <state_interface name="velocity">
-                <param name="initial_value">0.0</param>
-            </state_interface>
-            <state_interface name="position">
-                <param name="initial_value">0.0</param>
-            </state_interface>
-            <state_interface name="effort">
-                <param name="initial_value">0.0</param>
-            </state_interface>
+            <!-- Left Wheel Joint -->
+            <joint name="${prefix}left_wheel_joint">
+                <command_interface name="velocity">
+                    <param name="min">-1000</param>
+                    <param name="max">1000</param>
+                </command_interface>
+                <state_interface name="velocity">
+                    <param name="initial_value">0.0</param>
+                </state_interface>
+                <state_interface name="position">
+                    <param name="initial_value">0.0</param>
+                </state_interface>
             </joint>
-            <joint name="${prefix}rear_left_wheel_joint">
-            <param name="mimic">virtual_rear_wheel_joint</param>
-            <param name="multiplier">${speed_multiplier}</param>
-            <state_interface name="velocity">
-                <param name="initial_value">0.0</param>
-            </state_interface>
-            <state_interface name="position">
-                <param name="initial_value">0.0</param>
-            </state_interface>
-            <state_interface name="effort">
-                <param name="initial_value">0.0</param>
-            </state_interface>
-            </joint>
-            <joint name="${prefix}rear_right_wheel_joint">
-            <param name="mimic">virtual_rear_wheel_joint</param>
-            <param name="multiplier">${speed_multiplier}</param>
-            <state_interface name="velocity">
-                <param name="initial_value">0.0</param>
-            </state_interface>
-            <state_interface name="position">
-                <param name="initial_value">0.0</param>
-            </state_interface>
-            <state_interface name="effort">
-                <param name="initial_value">0.0</param>
-            </state_interface>
-            </joint>
-            <!-- steer joint -->
-            <joint name="${prefix}virtual_front_wheel_joint">
-            <command_interface name="position">
-                <param name="min">-1000</param>
-                <param name="max">1000</param>
-            </command_interface>
-            <state_interface name="position">
-                <param name="initial_value">0.0</param>
-            </state_interface>
-            <state_interface name="effort">
-                <param name="initial_value">0.0</param>
-            </state_interface>
-            </joint>
-            <joint name="${prefix}front_right_wheel_joint">
-            <param name="mimic">virtual_rear_wheel_joint</param>
-            <param name="multiplier">${speed_multiplier}</param>
-            <state_interface name="velocity">
-                <param name="initial_value">0.0</param>
-            </state_interface>
-            <state_interface name="position">
-                <param name="initial_value">0.0</param>
-            </state_interface>
-            <state_interface name="effort">
-                <param name="initial_value">0.0</param>
-            </state_interface>
-            </joint>
-            <joint name="${prefix}front_left_wheel_joint">
-            <param name="mimic">virtual_rear_wheel_joint</param>
-            <param name="multiplier">${speed_multiplier}</param>
-            <state_interface name="velocity">
-                <param name="initial_value">0.0</param>
-            </state_interface>
-            <state_interface name="position">
-                <param name="initial_value">0.0</param>
-            </state_interface>
-            <state_interface name="effort">
-                <param name="initial_value">0.0</param>
-            </state_interface>
-            </joint>
-            <joint name="${prefix}front_left_steer_joint">
-            <param name="mimic">virtual_front_wheel_joint</param>
-            <param name="multiplier">1</param>
-            <state_interface name="position">
-                <param name="initial_value">0.0</param>
-            </state_interface>
-            <state_interface name="effort">
-                <param name="initial_value">0.0</param>
-            </state_interface>
-            </joint>
-            <joint name="${prefix}front_right_steer_joint">
-            <param name="mimic">virtual_front_wheel_joint</param>
-            <param name="multiplier">1</param>
-            <state_interface name="position">
-                <param name="initial_value">0.0</param>
-            </state_interface>
-            <state_interface name="effort">
-                <param name="initial_value">0.0</param>
-            </state_interface>
+            <!-- Right Wheel Joint -->
+            <joint name="${prefix}right_wheel_joint">
+                <command_interface name="velocity">
+                    <param name="min">-1000</param>
+                    <param name="max">1000</param>
+                </command_interface>
+                <state_interface name="velocity">
+                    <param name="initial_value">0.0</param>
+                </state_interface>
+                <state_interface name="position">
+                    <param name="initial_value">0.0</param>
+                </state_interface>
             </joint>
         </ros2_control>

File: ros2_ws/src/robot_hardware/description/urdf/core.urdf.xacro (robot description, xacro)
@@ -4,6 +4,9 @@
   <xacro:arg name="prefix" default="" />
   <xacro:arg name="sim_mode" default="false"/>
-  <!-- Import Constants -->
+  <!-- Import Static Files -->
   <xacro:include filename="$(find robot_hardware)/urdf/util/constants.xacro" />
+  <!-- Import Macros -->
+  <xacro:include filename="$(find robot_hardware)/urdf/util/macros/wheel.xacro" />
+  <xacro:include filename="$(find robot_hardware)/urdf/util/macros/dead_wheel.xacro" />
   <!-- Import Robot Description -->
   <xacro:include filename="$(find robot_hardware)/urdf/robot.urdf.xacro" />
@@ -12,14 +15,5 @@
   <!-- Import Hardware Interface -->
   <xacro:include filename="$(find robot_hardware)/ros2_control/robot_hardware.ros2_control.xacro" />
-  <!-- <xacro:include filename="$(find robot_hardware)/ros2_control/sim.xacro"/> -->
-  <!-- Import Camera -->
-  <!-- <xacro:include filename="$(find robot_hardware)/urdf/components/camera.xacro" /> -->
-  <!-- Import Depth Camera -->
-  <!-- <xacro:include filename="$(find robot_hardware)/urdf/components/depth_camera.xacro" /> -->
-  <!-- Import LiDAR -->
-  <!-- <xacro:include filename="$(find robot_hardware)/urdf/components/lidar.xacro" /> -->
   <xacro:robot_hardware prefix="$(arg prefix)" />
-  <!-- <xacro:camera prefix="$(arg prefix)"/> -->
-  <!-- <xacro:lidar prefix="$(arg prefix)"/> -->
-  <xacro:robot_hardware_ros2_control name="RobotSystemHardware" prefix="$(arg prefix)" />
+  <xacro:robot_hardware_ros2_control name="RobotSystemHardware" prefix="$(arg prefix)"/>
 </robot>

File: ros2_ws/src/robot_hardware/description/urdf/robot.urdf.xacro (robot description, xacro)
@@ -2,14 +2,53 @@
 <robot xmlns:xacro="http://www.ros.org/wiki/xacro">
   <xacro:macro name="robot_hardware" params="prefix">
-    <!-- Base Link and Base Footprint -->
-    <xacro:include filename="$(find robot_hardware)/urdf/components/base.xacro" />
-    <!-- Chassis Link -->
-    <xacro:include filename="$(find robot_hardware)/urdf/components/chassis.xacro" />
-        <xacro:include filename="$(find robot_hardware)/urdf/macros/front_wheel.xacro" />
-        <xacro:include filename="$(find robot_hardware)/urdf/macros/rear_wheel.xacro" />
-        <xacro:front_wheel name="front_left" x="${wheel_x}" y="${wheel_y}" z="${wheel_z}" side="1"/>
-        <xacro:front_wheel name="front_right" x="${wheel_x}" y="${-wheel_y}" z="${wheel_z}" side="-1"/>
-        <xacro:rear_wheel name="rear_left" x="${-wheel_x}" y="${wheel_y}" z="${wheel_z}" side="1"/>
-        <xacro:rear_wheel name="rear_right" x="${-wheel_x}" y="${-wheel_y}" z="${wheel_z}" side="-1"/>
+    <!-- Base Link -->
+    <link name="${prefix}base_link"/>
+    <!-- Base Footprint -->
+    <link name="${prefix}base_footprint"/>
+    <!-- Chassis -->
+    <link name="${prefix}chassis_link">
+      <collision>
+        <origin xyz="0 0 0" rpy="0 0 ${PI/2}"/>
+        <geometry>
+          <mesh filename="file://$(find robot_hardware)/urdf/assets/chassis/Chassis.stl"/>
+        </geometry>
+      </collision>
+      <visual>
+        <origin xyz="0 0 0" rpy="0 0 ${PI/2}"/>
+        <geometry>
+          <mesh filename="file://$(find robot_hardware)/urdf/assets/chassis/Chassis.stl"/>
+        </geometry>
+        <cast_shadows>false</cast_shadows>
+        <material name="grey"/>
+      </visual>
+      <inertial>
+        <origin xyz="0 0 0" rpy="0 0 0"/>
+        <mass value="${base_mass}"/>
+          <inertia
+            ixx="${0.01952332}" ixy="0.0" ixz="0.0"
+            iyy="${0.01450326}" iyz="${-0.00000016}"
+            izz="${0.02678084}"/>
+        </inertial>
+    </link>
+    <gazebo reference="chassis_link">
+      <material>Gazebo/Grey</material>
+    </gazebo>
+    <joint name="${prefix}chassis_joint" type="fixed">
+      <parent link="${prefix}base_link"/>
+      <child link="${prefix}chassis_link"/>
+      <origin xyz="0 0 ${.0199 + wheel_radius}" rpy="0 0 ${PI}"/>
+      <axis xyz="0 0 1"/>
+      <dynamics damping="${damping}"/>
+    </joint>
+    <joint name="${prefix}base_footprint_joint" type="fixed">
+      <parent link="${prefix}base_link"/>
+      <child link="${prefix}base_footprint"/>
+      <origin xyz="0 0 0" rpy="0 0 0"/>
+    </joint>
+    <!--front is positive, left is positive-->
+    <xacro:wheel name="left" x="0" y="0" z="0" front="-1" side="-1"/>
+    <xacro:wheel name="right" x="0" y="0" z="0" front="-1" side="1"/>
+    <xacro:dead_wheel name="left_caster" x="0" y="0" z="0" front="1" side="-1"/>
+    <xacro:dead_wheel name="right_caster" x="0" y="0" z="0" front="1" side="1"/>
   </xacro:macro>
 </robot>

File: ros2_ws/src/robot_hardware/description/urdf/util/constants.xacro (robot description, xacro)
@@ -1,21 +1,15 @@
 <?xml version="1.0"?>
 <robot xmlns:xacro="http://www.ros.org/wiki/xacro">
-    <!-- Physics Constants -->
-        <xacro:property name="PI" value="3.1415926535897931"/>
-        <xacro:property name="friction" value="1"/>
-        <xacro:property name="min_depth" value="0.5"/>
-        <xacro:property name="damping" value="0.001"/>
-    <!-- System Wide Constants -->
-        <xacro:property name="chassis_mass" value="20" /> <!-- arbitrary value for chassis mass -->
-    <!-- Mechanism Specific -->
-        <!-- Wheels -->
-            <xacro:property name="track_width" value="0.165" />
-            <xacro:property name="track_length" value="0.18" />
-            <xacro:property name="wheel_width" value="0.03" />
-            <xacro:property name="wheel_radius" value="0.03725" />
-            <xacro:property name="wheel_mass" value="0.5" /> <!-- arbitrary value for wheel mass -->
-            <!-- Remember to switch X and Y for onshape to ros -->
-            <xacro:property name="wheel_x" value="0.09"/>
-            <xacro:property name="wheel_y" value="0.0675"/>
-            <xacro:property name="wheel_z" value="0.02"/>
+    <xacro:property name="PI" value="3.1415926535897931"/>
+    <xacro:property name="base_mass" value="4" /> <!-- arbitrary value for base mass -->
+    <xacro:property name="base_width" value="0.240" />
+    <xacro:property name="base_length" value="0.300" />
+    <xacro:property name="base_height" value="0.140" />
+    <xacro:property name="wheelbase" value=".2845" />
+    <xacro:property name="wheel_width" value="0.0265" />
+    <xacro:property name="wheel_radius" value="0.032" />
+    <xacro:property name="wheel_mass" value="0.34055" /> <!-- arbitrary value for wheel mass -->
+    <xacro:property name="friction" value="10"/>
+    <xacro:property name="min_depth" value="0.5"/>
+    <xacro:property name="damping" value="0.001"/>
 </robot>
